File: keyboard.kicad_pcb (KiCad board)
At the start: 2 copper layers, 285 x 94.6 mm, 257 parts, among them J1 USB_B_Micro, SW1 SW_Push

Commit message: WIP
Parts:
- removed D39, D40, D41, D42, D43, D44, D45, D46, D47, D48, D49, D50, D51, D52, D53, D54, D55, D56, D57, D58, D59, D60, D61, D62, D63, D64, D65: 1N4148, 0805:0805D
- removed the LED3 at (78.6, 111.9)
- added C1: 1uF, Capacitor_SMD:C_0603_1608Metric, B.Cu at (225.9, 178.6)
- added C2: 1uF, Capacitor_SMD:C_0603_1608Metric, B.Cu at (231.3, 178.3)
- added C3: 1uF, Capacitor_SMD:C_0603_1608Metric, B.Cu at (136.7, 148.7)
- added C4: 1uF, Capacitor_SMD:C_0603_1608Metric, B.Cu at (135.9, 143.4)
- added C6: 1uF, Capacitor_SMD:C_0603_1608Metric, F.Cu at (81.3, 62.2)
- added J2: JST_PH, Connector_JST:JST_PH_S2B-PH-K_1x02_P2.00mm_Horizontal, B.Cu at (206.4, 102.2)
- added J3: Conn_ARM_JTAG_SWD_10, swd:PinHeader_2x05_P1.27mm_Vertical_SMD, F.Cu at (221.0, 149.9)
- added J4: Conn_01x08, Connector_PinHeader_2.54mm:PinHeader_1x08_P2.54mm_Vertical, F.Cu at (164.4, 170.7)
- added LED85: LED, LED_SMD:LED_0805_2012Metric, B.Cu at (74.9, 67.1)
- added Q1: PMOS, Package_TO_SOT_SMD:SOT-23, F.Cu at (193.0, 170.5)
- added Q2: PMOS, Package_TO_SOT_SMD:SOT-23, F.Cu at (167.9, 173.7)
- added R1: R, Resistor_SMD:R_0603_1608Metric, B.Cu at (226.7, 181.6)
- added R10: R, Resistor_THT:R_Axial_DIN0207_L6.3mm_D2.5mm_P10.16mm_Horizontal, F.Cu at (167.3, 170.4)
- added R2: 10k, Resistor_SMD:R_0603_1608Metric, B.Cu at (229.1, 173.5)
- added R3: R, Resistor_SMD:R_0603_1608Metric, B.Cu at (75.6, 71.1)
- added R4: 10k, Resistor_SMD:R_0603_1608Metric, F.Cu at (183.5, 172.7)
- added R5: 1.5k, Resistor_SMD:R_0603_1608Metric, F.Cu at (193.0, 173.0)
- added R6: 10k, Resistor_SMD:R_0603_1608Metric, F.Cu at (177.6, 172.7)
- added R7: 10k, Resistor_SMD:R_0603_1608Metric, F.Cu at (180.6, 172.7)
- added R8: R, Resistor_SMD:R_0603_1608Metric, F.Cu at (174.6, 172.7)
- added R9: R, Resistor_THT:R_Axial_DIN0207_L6.3mm_D2.5mm_P10.16mm_Horizontal, F.Cu at (179.6, 170.4)
- added SW2: SSSS912000, switch:SSSS912000, B.Cu at (90.2, 113.0)
- added U1: BL652, RF_Module:Laird_BL652, B.Cu at (170.2, 151.1)
- added U2: BQ21040, Package_TO_SOT_SMD:SOT-23-6, B.Cu at (228.6, 179.1)
- added U3: TLV70033, Package_TO_SOT_SMD:SOT-23-5, B.Cu at (135.9, 146.1)
- D1, D14, D23, D26, D29, D32, D35, D4, D7: value 1N4148 -> D; footprint 0805:0805D -> Diode_SMD:D_SOT-23_ANK
- D10, D11, D12, D13, D15, D16, D17, D18, D19, D2, D20, D21, D22, D24, D25, D27, D28, D3, D30, D31, D33, D34, D36, D37, D5, D6, D8, D9: value 1N4148 -> D_x2_KCom_AAK; footprint 0805:0805D -> Package_TO_SOT_SMD:SOT-23
- D38: value 1N4148 -> D; footprint 0805:0805D -> Diode_SMD:D_0805_2012Metric; moved to F.Cu
- SW1: moved to F.Cu
- moved D23 191.4 mm to (335.3, 82.5)
- moved D36 131.4 mm to (325.1, 84.5)
- moved D29 129.4 mm to (294.6, 139.7)
- moved D32 118.6 mm to (303.5, 142.2), turned to 180 degrees
- moved D27 112.4 mm to (271.8, 82.5)
- moved D35 112.3 mm to (322.6, 142.2), turned to 180 degrees
- moved D37 111.2 mm to (321.3, 120.7)
- moved D33 110.6 mm to (309.9, 82.5)
- moved D26 102.9 mm to (275.6, 139.7)
- moved D30 101.9 mm to (290.8, 82.5)
- moved D31 100.1 mm to (294.6, 121.9)
- moved D34 98.7 mm to (304.8, 120.7), turned to 180 degrees
- moved D19 94.9 mm to (214.6, 82.5)
- moved D38 94.4 mm to (171.4, 173.0)
- moved D24 90.6 mm to (252.7, 82.5)
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- renumbered LED11 to LED10, LED12 to LED11, LED13 to LED12, LED14 to LED13, LED15 to LED14, LED16 to LED15, LED17 to LED16, LED18 to LED17, LED19 to LED18, LED20 to LED19, LED21 to LED20, LED22 to LED21, LED23 to LED22, LED24 to LED23, LED25 to LED24, LED26 to LED25, LED27 to LED26, LED28 to LED27, LED29 to LED28, LED30 to LED29, LED4 to LED3, LED31 to LED30, LED32 to LED31, LED33 to LED32, LED34 to LED33, LED35 to LED34, LED36 to LED35, LED37 to LED36, LED38 to LED37, LED39 to LED38, LED40 to LED39, LED5 to LED4, LED41 to LED40, LED42 to LED41, LED43 to LED42, LED44 to LED43, LED45 to LED44, LED46 to LED45, LED47 to LED46, LED48 to LED47, LED49 to LED48, LED50 to LED49, LED6 to LED5, LED51 to LED50, LED52 to LED51, LED53 to LED52, LED54 to LED53, LED55 to LED54, LED56 to LED55, LED57 to LED56, LED58 to LED57, LED59 to LED58, LED60 to LED59, LED7 to LED6, LED61 to LED60, LED62 to LED61, LED63 to LED62, LED64 to LED63, LED65 to LED64, LED66 to LED65, LED67 to LED66, LED68 to LED67, LED69 to LED68, LED70 to LED69, LED8 to LED7, LED71 to LED70, LED72 to LED71, LED73 to LED72, LED74 to LED73, LED75 to LED74, LED76 to LED75, LED77 to LED76, LED78 to LED77, LED79 to LED78, LED80 to LED79, LED9 to LED8, LED81 to LED80, LED82 to LED81, LED83 to LED82, LED84 to LED83, LED85 to LED84, LED10 to LED9, S36 to S34, S34 to S35, S35 to S36
Connections:
- net /Leds/CAPS_LED- renamed /Leds/CAPS_LED+
- net Net-(J1-Pad3) renamed /USB_D+
- D10 pad 1: /col2 -> Net-(D10-Pad1)
- D11 pad 1: /col3 -> Net-(D11-Pad1)
- D12 pad 1: /col3 -> Net-(D12-Pad1)
- D13 pad 1: /col3 -> Net-(D13-Pad1)
- D14 pad 1: /col3 -> /col6
- D15 pad 1: /col3 -> Net-(D15-Pad1)
- D16 pad 1: /col4 -> Net-(D16-Pad1)
- D17 pad 1: /col4 -> Net-(D17-Pad1)
- D18 pad 1: /col4 -> Net-(D18-Pad1)
- D19 pad 1: /col4 -> Net-(D19-Pad1)
- D2 pad 1: /col1 -> Net-(D2-Pad1)
- D20 pad 1: /col5 -> Net-(D20-Pad1)
- D21 pad 1: /col5 -> Net-(D21-Pad1)
- D22 pad 1: /col5 -> Net-(D22-Pad1)
- D23 pad 1: /col5 -> /col10
- D24 pad 1: /col6 -> Net-(D24-Pad1)
- D25 pad 1: /col6 -> Net-(D25-Pad1)
- D26 pad 1: /col6 -> /col11
- D27 pad 1: /col6 -> Net-(D27-Pad1)
- D28 pad 1: /col6 -> Net-(D28-Pad1)
- D29 pad 1: /col7 -> /col12
- D3 pad 1: /col1 -> Net-(D3-Pad1)
- D30 pad 1: /col7 -> Net-(D30-Pad1)
- D31 pad 1: /col7 -> Net-(D31-Pad1)
- D32 pad 1: /col7 -> /col13
- D33 pad 1: /col8 -> Net-(D33-Pad1)
- D34 pad 1: /col8 -> Net-(D34-Pad1)
- D35 pad 1: /col8 -> /col14
- D36 pad 1: /col8 -> Net-(D36-Pad1)
- D37 pad 1: /col9 -> Net-(D37-Pad1)
- D38 pad 1: /col9 -> /VBAT
- D38 pad 2: Net-(D38-Pad2) -> /VBUS
- D4 pad 1: /col1 -> /col2
- D5 pad 1: /col1 -> Net-(D5-Pad1)
- D6 pad 1: /col2 -> Net-(D6-Pad1)
- D7 pad 1: /col2 -> /col3
- D8 pad 1: /col2 -> Net-(D8-Pad1)
- D9 pad 1: /col2 -> Net-(D9-Pad1)
- J1 pad 1: Net-(J1-Pad1) -> /VBUS
- J1 pad 2: Net-(J1-Pad2) -> /USB_D-
- J1 pad 5: Net-(J1-Pad5) -> GND
- J1 pad 6: Net-(J1-Pad5) -> Net-(J1-Pad6)
- LED1 pad 2: /Leds/LED+ -> /CAPS_LED
- LED10 pad 1: /Leds/LED- -> /Leds/LED+
- LED10 pad 2: /Leds/LED+ -> GND
- LED11 pad 1: /Leds/LED- -> /Leds/LED+
- LED11 pad 2: /Leds/LED+ -> GND
- LED12 pad 1: /Leds/LED- -> /Leds/LED+
- LED12 pad 2: /Leds/LED+ -> GND
- LED13 pad 1: /Leds/LED- -> /Leds/LED+
- LED13 pad 2: /Leds/LED+ -> GND
- LED14 pad 1: /Leds/LED- -> GND
- LED15 pad 1: /Leds/LED- -> GND
- LED16 pad 1: /Leds/LED- -> /Leds/LED+
- LED16 pad 2: /Leds/LED+ -> GND
- LED17 pad 1: /Leds/LED- -> /Leds/LED+
- LED17 pad 2: /Leds/LED+ -> GND
- LED18 pad 1: /Leds/LED- -> /Leds/LED+
- LED18 pad 2: /Leds/LED+ -> GND
- LED19 pad 1: /Leds/LED- -> /Leds/LED+
- LED19 pad 2: /Leds/LED+ -> GND
- LED2 pad 2: /Leds/LED+ -> /CAPS_LED
- LED20 pad 1: /Leds/LED- -> /Leds/LED+
- LED20 pad 2: /Leds/LED+ -> GND
- LED21 pad 1: /Leds/LED- -> GND
- LED22 pad 1: /Leds/LED- -> /Leds/LED+
- LED22 pad 2: /Leds/LED+ -> GND
- LED23 pad 1: /Leds/LED- -> /Leds/LED+
- LED23 pad 2: /Leds/LED+ -> GND
- LED24 pad 1: /Leds/LED- -> /Leds/LED+
- LED24 pad 2: /Leds/LED+ -> GND
- LED25 pad 1: /Leds/LED- -> /Leds/LED+
- LED25 pad 2: /Leds/LED+ -> GND
- LED26 pad 1: /Leds/LED- -> /Leds/LED+
- LED26 pad 2: /Leds/LED+ -> GND
- LED27 pad 1: /Leds/LED- -> /Leds/LED+
- LED27 pad 2: /Leds/LED+ -> GND
- LED28 pad 1: /Leds/LED- -> /Leds/LED+
- LED28 pad 2: /Leds/LED+ -> GND
- LED29 pad 1: /Leds/LED- -> /Leds/LED+
- LED29 pad 2: /Leds/LED+ -> GND
- LED3 pad 1: /Leds/LED- -> /Leds/LED+
- LED3 pad 2: /Leds/LED+ -> GND
- LED30 pad 1: /Leds/LED- -> /Leds/LED+
- LED30 pad 2: /Leds/LED+ -> GND
- LED31 pad 1: /Leds/LED- -> /Leds/LED+
- LED31 pad 2: /Leds/LED+ -> GND
- LED32 pad 1: /Leds/LED- -> /Leds/LED+
- LED32 pad 2: /Leds/LED+ -> GND
- LED33 pad 1: /Leds/LED- -> /Leds/LED+
- LED33 pad 2: /Leds/LED+ -> GND
- LED34 pad 1: /Leds/LED- -> /Leds/LED+
- LED34 pad 2: /Leds/LED+ -> GND
- LED35 pad 1: /Leds/LED- -> /Leds/LED+
- LED35 pad 2: /Leds/LED+ -> GND
- LED36 pad 1: /Leds/LED- -> /Leds/LED+
- LED36 pad 2: /Leds/LED+ -> GND
- LED37 pad 1: /Leds/LED- -> /Leds/LED+
- LED37 pad 2: /Leds/LED+ -> GND
- LED38 pad 1: /Leds/LED- -> /Leds/LED+
- LED38 pad 2: /Leds/LED+ -> GND
- LED39 pad 1: /Leds/LED- -> /Leds/LED+
- LED39 pad 2: /Leds/LED+ -> GND
- LED4 pad 1: /Leds/LED- -> /Leds/LED+
- LED4 pad 2: /Leds/LED+ -> GND
- LED40 pad 1: /Leds/LED- -> /Leds/LED+
- LED40 pad 2: /Leds/LED+ -> GND
- LED41 pad 1: /Leds/LED- -> /Leds/LED+
- LED41 pad 2: /Leds/LED+ -> GND
- LED42 pad 1: /Leds/LED- -> /Leds/LED+
- LED42 pad 2: /Leds/LED+ -> GND
- LED43 pad 1: /Leds/LED- -> /Leds/LED+
- LED43 pad 2: /Leds/LED+ -> GND
- LED44 pad 1: /Leds/LED- -> /Leds/LED+
- LED44 pad 2: /Leds/LED+ -> GND
- LED45 pad 1: /Leds/LED- -> /Leds/LED+
- LED45 pad 2: /Leds/LED+ -> GND
- LED46 pad 1: /Leds/LED- -> /Leds/LED+
- LED46 pad 2: /Leds/LED+ -> GND
- LED47 pad 1: /Leds/LED- -> /Leds/LED+
- LED47 pad 2: /Leds/LED+ -> GND
- LED48 pad 1: /Leds/LED- -> /Leds/LED+
- LED48 pad 2: /Leds/LED+ -> GND
- LED49 pad 1: /Leds/LED- -> /Leds/LED+
- LED49 pad 2: /Leds/LED+ -> GND
- LED5 pad 1: /Leds/LED- -> /Leds/LED+
- LED5 pad 2: /Leds/LED+ -> GND
- LED50 pad 1: /Leds/LED- -> /Leds/LED+
- LED50 pad 2: /Leds/LED+ -> GND
- LED51 pad 1: /Leds/LED- -> /Leds/LED+
- LED51 pad 2: /Leds/LED+ -> GND
- LED52 pad 1: /Leds/LED- -> /Leds/LED+
- LED52 pad 2: /Leds/LED+ -> GND
- LED53 pad 1: /Leds/LED- -> /Leds/LED+
- LED53 pad 2: /Leds/LED+ -> GND
- LED54 pad 1: /Leds/LED- -> /Leds/LED+
- LED54 pad 2: /Leds/LED+ -> GND
- LED55 pad 1: /Leds/LED- -> /Leds/LED+
- LED55 pad 2: /Leds/LED+ -> GND
- LED56 pad 1: /Leds/LED- -> /Leds/LED+
- LED56 pad 2: /Leds/LED+ -> GND
- LED57 pad 1: /Leds/LED- -> /Leds/LED+
- LED57 pad 2: /Leds/LED+ -> GND
- LED58 pad 1: /Leds/LED- -> /Leds/LED+
- LED58 pad 2: /Leds/LED+ -> GND
- LED59 pad 1: /Leds/LED- -> GND
- LED6 pad 1: /Leds/LED- -> /Leds/LED+
- LED6 pad 2: /Leds/LED+ -> GND
- LED60 pad 1: /Leds/LED- -> /Leds/LED+
- LED60 pad 2: /Leds/LED+ -> GND
- LED61 pad 1: /Leds/LED- -> /Leds/LED+
- LED61 pad 2: /Leds/LED+ -> GND
- LED62 pad 1: /Leds/LED- -> /Leds/LED+
- LED62 pad 2: /Leds/LED+ -> GND
- LED63 pad 1: /Leds/LED- -> /Leds/LED+
- LED63 pad 2: /Leds/LED+ -> GND
- LED64 pad 1: /Leds/LED- -> GND
- LED65 pad 1: /Leds/LED- -> GND
- LED66 pad 1: /Leds/LED- -> /Leds/LED+
- LED66 pad 2: /Leds/LED+ -> GND
- LED67 pad 1: /Leds/LED- -> /Leds/LED+
- LED67 pad 2: /Leds/LED+ -> GND
- LED68 pad 1: /Leds/LED- -> /Leds/LED+
- LED68 pad 2: /Leds/LED+ -> GND
- LED69 pad 1: /Leds/LED- -> /Leds/LED+
- LED69 pad 2: /Leds/LED+ -> GND
- LED7 pad 1: /Leds/LED- -> /Leds/LED+
- LED7 pad 2: /Leds/LED+ -> GND
- LED70 pad 1: /Leds/LED- -> /Leds/LED+
- LED70 pad 2: /Leds/LED+ -> GND
- LED71 pad 1: /Leds/LED- -> /Leds/LED+
- LED71 pad 2: /Leds/LED+ -> GND
- LED72 pad 1: /Leds/LED- -> /Leds/LED+
- LED72 pad 2: /Leds/LED+ -> GND
- LED73 pad 1: /Leds/LED- -> GND
- LED74 pad 1: /Leds/LED- -> /Leds/LED+
- LED74 pad 2: /Leds/LED+ -> GND
- LED75 pad 1: /Leds/LED- -> /Leds/LED+
- LED75 pad 2: /Leds/LED+ -> GND
- LED76 pad 1: /Leds/LED- -> /Leds/LED+
- LED76 pad 2: /Leds/LED+ -> GND
- LED77 pad 1: /Leds/LED- -> /Leds/LED+
- LED77 pad 2: /Leds/LED+ -> GND
- LED78 pad 1: /Leds/LED- -> /Leds/LED+
- LED78 pad 2: /Leds/LED+ -> GND
- LED79 pad 1: /Leds/LED- -> /Leds/LED+
- LED79 pad 2: /Leds/LED+ -> GND
- LED8 pad 1: /Leds/LED- -> GND
- LED80 pad 1: /Leds/LED- -> /Leds/LED+
- LED80 pad 2: /Leds/LED+ -> GND
- LED81 pad 1: /Leds/LED- -> /Leds/LED+
- LED81 pad 2: /Leds/LED+ -> GND
- LED82 pad 1: /Leds/LED- -> /Leds/LED+
- LED82 pad 2: /Leds/LED+ -> GND
- LED83 pad 1: /Leds/LED- -> /Leds/LED+
- LED83 pad 2: /Leds/LED+ -> GND
- LED84 pad 1: /Leds/LED- -> GND
- LED9 pad 1: /Leds/LED- -> /Leds/LED+
- LED9 pad 2: /Leds/LED+ -> GND
- S1 pad 2: Net-(D1-Pad2) -> Net-(D2-Pad1)
- S10 pad 2: Net-(D7-Pad2) -> Net-(D5-Pad1)
- S11 pad 2: Net-(D8-Pad2) -> Net-(D6-Pad2)
- S12 pad 2: Net-(D9-Pad2) -> Net-(D6-Pad1)
- S13 pad 2: Net-(D10-Pad2) -> Net-(D4-Pad2)
- S14 pad 1: Net-(D10-Pad2) -> Net-(D4-Pad2)
- S15 pad 2: Net-(D10-Pad2) -> Net-(D4-Pad2)
- S16 pad 2: Net-(D11-Pad2) -> Net-(D8-Pad2)
- S17 pad 2: Net-(D12-Pad2) -> Net-(D8-Pad1)
- S18 pad 2: Net-(D13-Pad2) -> Net-(D9-Pad2)
- S19 pad 2: Net-(D14-Pad2) -> Net-(D9-Pad1)
- S20 pad 2: Net-(D15-Pad2) -> Net-(D7-Pad2)
- S21 pad 2: Net-(D15-Pad2) -> Net-(D7-Pad2)
- S22 pad 2: Net-(D16-Pad2) -> Net-(D10-Pad2)
- S23 pad 2: Net-(D17-Pad2) -> Net-(D10-Pad1)
- S24 pad 2: Net-(D18-Pad2) -> Net-(D11-Pad2)
- S25 pad 2: Net-(D19-Pad2) -> Net-(D11-Pad1)
- S26 pad 2: Net-(D20-Pad2) -> Net-(D12-Pad2)
- S27 pad 2: Net-(D21-Pad2) -> Net-(D12-Pad1)
- S28 pad 2: Net-(D22-Pad2) -> Net-(D13-Pad2)
- S29 pad 2: Net-(D23-Pad2) -> Net-(D13-Pad1)
- S3 pad 2: Net-(D3-Pad2) -> Net-(D3-Pad1)
- S30 pad 2: Net-(D24-Pad2) -> Net-(D15-Pad2)
- S31 pad 2: Net-(D25-Pad2) -> Net-(D15-Pad1)
- S32 pad 2: Net-(D26-Pad2) -> Net-(D16-Pad2)
- S33 pad 2: Net-(D27-Pad2) -> Net-(D16-Pad1)
- S34 pad 2: Net-(D28-Pad2) -> Net-(D14-Pad2)
- S35 pad 2: Net-(D28-Pad2) -> Net-(D14-Pad2)
- S36 pad 2: Net-(D28-Pad2) -> Net-(D14-Pad2)
- S37 pad 2: Net-(D29-Pad2) -> Net-(D17-Pad2)
- S38 pad 2: Net-(D30-Pad2) -> Net-(D17-Pad1)
- S39 pad 2: Net-(D31-Pad2) -> Net-(D18-Pad2)
- S4 pad 2: Net-(D3-Pad2) -> Net-(D3-Pad1)
- S40 pad 2: Net-(D32-Pad2) -> Net-(D18-Pad1)
- S41 pad 2: Net-(D33-Pad2) -> Net-(D19-Pad2)
- S42 pad 2: Net-(D34-Pad2) -> Net-(D19-Pad1)
- S43 pad 2: Net-(D35-Pad2) -> Net-(D20-Pad2)
- S44 pad 2: Net-(D36-Pad2) -> Net-(D20-Pad1)
- S45 pad 2: Net-(D37-Pad2) -> Net-(D21-Pad2)
- S46 pad 2: Net-(D38-Pad2) -> Net-(D21-Pad1)
- S47 pad 2: Net-(D39-Pad2) -> Net-(D22-Pad2)
- S48 pad 2: Net-(D40-Pad2) -> Net-(D22-Pad1)
- S49 pad 2: Net-(D41-Pad2) -> Net-(D24-Pad2)
- S5 pad 2: Net-(D4-Pad2) -> Net-(D3-Pad2)
- S50 pad 2: Net-(D42-Pad2) -> Net-(D24-Pad1)
- S51 pad 2: Net-(D43-Pad2) -> Net-(D25-Pad2)
- S52 pad 2: Net-(D44-Pad2) -> Net-(D25-Pad1)
- S53 pad 2: Net-(D45-Pad2) -> Net-(D23-Pad2)
- S54 pad 2: Net-(D46-Pad2) -> Net-(D27-Pad2)
- S55 pad 2: Net-(D47-Pad2) -> Net-(D27-Pad1)
- S56 pad 2: Net-(D48-Pad2) -> Net-(D28-Pad2)
- S57 pad 2: Net-(D49-Pad2) -> Net-(D28-Pad1)
- S58 pad 2: Net-(D50-Pad2) -> Net-(D26-Pad2)
- S59 pad 2: Net-(D50-Pad2) -> Net-(D26-Pad2)
- S6 pad 2: Net-(D4-Pad2) -> Net-(D3-Pad2)
- S60 pad 2: Net-(D51-Pad2) -> Net-(D30-Pad2)
- S61 pad 2: Net-(D52-Pad2) -> Net-(D30-Pad1)
- S62 pad 2: Net-(D53-Pad2) -> Net-(D31-Pad2)
- S63 pad 2: Net-(D54-Pad2) -> Net-(D31-Pad1)
- S64 pad 2: Net-(D55-Pad2) -> Net-(D29-Pad2)
- S65 pad 2: Net-(D55-Pad2) -> Net-(D29-Pad2)
- S66 pad 2: Net-(D55-Pad2) -> Net-(D29-Pad2)
- S67 pad 2: Net-(D56-Pad2) -> Net-(D33-Pad2)
- S68 pad 2: Net-(D57-Pad2) -> Net-(D33-Pad1)
- S69 pad 2: Net-(D58-Pad2) -> Net-(D34-Pad1)
- S7 pad 2: Net-(D5-Pad2) -> Net-(D1-Pad2)
- S70 pad 2: Net-(D59-Pad2) -> Net-(D34-Pad2)
- S71 pad 2: Net-(D59-Pad2) -> Net-(D34-Pad2)
- S72 pad 2: Net-(D60-Pad2) -> Net-(D32-Pad2)
- S73 pad 2: Net-(D60-Pad2) -> Net-(D32-Pad2)
- S74 pad 2: Net-(D61-Pad2) -> Net-(D36-Pad2)
- S75 pad 2: Net-(D61-Pad2) -> Net-(D36-Pad2)
- S76 pad 2: Net-(D62-Pad2) -> Net-(D36-Pad1)
- S77 pad 2: Net-(D63-Pad2) -> Net-(D37-Pad2)
- S78 pad 2: Net-(D63-Pad2) -> Net-(D37-Pad2)
- S79 pad 2: Net-(D63-Pad2) -> Net-(D37-Pad2)
- S8 pad 2: Net-(D5-Pad2) -> Net-(D1-Pad2)
- S80 pad 2: Net-(D64-Pad2) -> Net-(D37-Pad1)
- S81 pad 1: Net-(D64-Pad2) -> Net-(D37-Pad1)
- S82 pad 2: Net-(D64-Pad2) -> Net-(D37-Pad1)
- S83 pad 2: Net-(D65-Pad2) -> Net-(D35-Pad2)
- S84 pad 2: Net-(D65-Pad2) -> Net-(D35-Pad2)
- S9 pad 2: Net-(D6-Pad2) -> Net-(D5-Pad2)
Routing:
- added copper zone on B.Cu, net /VBAT
- added copper zone on F.Cu, net /VBAT
- added copper zone on B.Cu, net /VBUS
- added copper zone on F.Cu, net /VBUS
- added copper zone on B.Cu, net GND
- removed copper zone on B.Cu, net (none)
Other:
- net class Default: trace_width 0.4064 -> 0.2032; via_dia 1 -> 0.6
- net class GND added: clearance 0.2032, trace_width 0.4064, via_dia 0.6, via_drill 0.4
- net class POWER: trace_width 0.508 -> 0.4064; via_dia 1 -> 0.8
- rule pad_to_mask_clearance: 0.1016 -> 0
- rule trace_min: 0.2032 -> 0.2
- rule via_min_size: 1 -> 0.6
- board text removed: "Fn"

Commit message: WIP
Parts:
- SW1: moved to B.Cu
- SW2: moved to F.Cu
- turned LED1 to 180 degrees
- turned LED10 to 180 degrees
- turned LED11 to 180 degrees
- turned LED12 to 180 degrees
- turned LED13 to 180 degrees
- turned LED14 to 180 degrees
- turned LED15 to 180 degrees
- turned LED16 to 180 degrees
- turned LED17 to 180 degrees
- turned LED18 to 180 degrees
- turned LED19 to 180 degrees
- turned LED2 to 180 degrees
- turned LED20 to 180 degrees
- turned LED21 to 180 degrees
- turned LED22 to 180 degrees
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
Commit message: WIP
Parts:
- removed the C1 at (225.9, 178.6)
- removed D5: D_x2_KCom_AAK, Package_TO_SOT_SMD:SOT-23
- removed the R1 at (226.7, 181.6)
- removed the SW1 at (91.4, 112.8)
- added C3: 1uF, Capacitor_SMD:C_0603_1608Metric, B.Cu at (237.6, 148.4)
- added D104: D_x2_KCom_AAK, Package_TO_SOT_SMD:SOT-23, B.Cu at (98.6, 79.2)
- added R3: R, Resistor_SMD:R_0603_1608Metric, B.Cu at (233.0, 151.8)
- C1: renamed from C6; moved to B.Cu
- D1: renamed from D38; moved to B.Cu
- J3: value Conn_ARM_JTAG_SWD_10 -> Conn_01x10; footprint swd:PinHeader_2x05_P1.27mm_Vertical_SMD -> Connector_PinHeader_2.54mm:PinHeader_1x10_P2.54mm_Vertical
- J4: value Conn_01x08 -> Conn_ARM_JTAG_SWD_10; footprint Connector_PinHeader_2.54mm:PinHeader_1x08_P2.54mm_Vertical -> swd:PinHeader_2x05_P1.27mm_Vertical_SMD
- Q1, Q2, R6, R7, R8: moved to B.Cu
- R1: renamed from R4; moved to B.Cu
- R10: footprint Resistor_THT:R_Axial_DIN0207_L6.3mm_D2.5mm_P10.16mm_Horizontal -> Resistor_SMD:R_0603_1608Metric; moved to B.Cu
- R2: renamed from R5; moved to B.Cu
- SW1: renamed from SW2; moved to B.Cu
- moved R10 120.7 mm to (67.3, 102.9), turned to 270 degrees
- moved R7 100.9 mm to (95.0, 119.4), turned to 270 degrees
- moved R6 100.0 mm to (95.0, 116.3), turned to 270 degrees
- moved R9 94.3 mm to (86.4, 156.2), turned to 90 degrees
- moved R8 91.0 mm to (88.9, 142.2), turned to 90 degrees
- moved Q2 87.4 mm to (86.4, 142.2), turned to 180 degrees
- moved D1 75.7 mm to (238.1, 137.2), turned to 270 degrees
- moved R2 64.2 mm to (136.4, 142.7)
- moved Q1 62.0 mm to (136.4, 145.3), turned to 90 degrees
- moved J4 61.2 mm to (221.0, 147.3), turned to 90 degrees
- moved R1 53.3 mm to (136.4, 147.8)
- moved C4 51.1 mm to (111.3, 104.4)
- moved C5 51.1 mm to (110.5, 99.1)
- moved U3 51.1 mm to (110.5, 101.7)
- moved R4 30.5 mm to (235.4, 143.6)
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- renumbered C3 to C4, C4 to C5, D2 to D101, D3 to D102, D1 to D103, D6 to D105, D4 to D106, D8 to D107, D9 to D108, D7 to D109, D10 to D110, D11 to D111, D12 to D112, D13 to D113, D15 to D114, D16 to D115, D14 to D116, D17 to D117, D18 to D118, D19 to D119, D20 to D120, D21 to D121, D22 to D122, D24 to D123, D25 to D124, D23 to D125, D27 to D126, D28 to D127, D26 to D128, D30 to D129, D31 to D130, D29 to D131, D33 to D132, D34 to D133, D32 to D134, D36 to D135, D37 to D136, D35 to D137, LED85 to LED1, LED1 to LED101, LED2 to LED102, LED3 to LED103, LED4 to LED104, LED5 to LED105, LED6 to LED106, LED7 to LED107, LED8 to LED108, LED9 to LED109, LED10 to LED110, LED11 to LED111, LED12 to LED112, LED13 to LED113, LED14 to LED114, LED15 to LED115, LED16 to LED116, LED17 to LED117, LED18 to LED118, LED19 to LED119, LED20 to LED120, LED21 to LED121, LED22 to LED122, LED23 to LED123, LED24 to LED124, LED25 to LED125, LED26 to LED126, LED27 to LED127, LED28 to LED128, LED29 to LED129, LED30 to LED130, LED31 to LED131, LED32 to LED132, LED33 to LED133, LED34 to LED134, LED35 to LED135, LED36 to LED136, LED37 to LED137, LED38 to LED138, LED39 to LED139, LED40 to LED140, LED41 to LED141, LED42 to LED142, LED43 to LED143, LED44 to LED144, LED45 to LED145, LED46 to LED146, LED47 to LED147, LED48 to LED148, LED49 to LED149, LED50 to LED150, LED51 to LED151, LED52 to LED152, LED54 to LED153, LED55 to LED154, LED56 to LED155, LED57 to LED156, LED58 to LED157, LED59 to LED158, LED60 to LED159, LED61 to LED160, LED62 to LED161, LED63 to LED162, LED64 to LED163, LED65 to LED164, LED66 to LED165, LED67 to LED166, LED68 to LED167, LED69 to LED168, LED70 to LED169, LED71 to LED170, LED72 to LED171, LED73 to LED172, LED74 to LED173, LED75 to LED174, LED76 to LED175, LED77 to LED176, LED78 to LED177, LED79 to LED178, LED80 to LED179, LED81 to LED180, LED82 to LED181, LED83 to LED182, LED84 to LED183, LED53 to LED184, R2 to R4, R3 to R5, S1 to S101, S2 to S102, S3 to S103, S4 to S104, S5 to S105, S6 to S106, S7 to S107, S8 to S108, S9 to S109, S10 to S110, S11 to S111, S12 to S112, S13 to S113, S14 to S114, S15 to S115, S16 to S116, S17 to S117, S18 to S118, S19 to S119, S20 to S120, S21 to S121, S22 to S122, S23 to S123, S24 to S124, S25 to S125, S26 to S126, S27 to S127, S28 to S128, S29 to S129, S30 to S130, S31 to S131, S32 to S132, S33 to S133, S34 to S134, S35 to S135, S36 to S136, S37 to S137, S38 to S138, S39 to S139, S40 to S140, S41 to S141, S42 to S142, S43 to S143, S44 to S144, S45 to S145, S46 to S146, S47 to S147, S48 to S148, S49 to S149, S50 to S150, S51 to S151, S52 to S152, S53 to S153, S54 to S154, S55 to S155, S56 to S156, S57 to S157, S58 to S158, S59 to S159, S60 to S160, S61 to S161, S62 to S162, S63 to S163, S64 to S164, S65 to S165, S66 to S166, S67 to S167, S68 to S168, S69 to S169, S70 to S170, S71 to S171, S72 to S172, S73 to S173, S74 to S174, S75 to S175, S76 to S176, S77 to S177, S78 to S178, S79 to S179, S80 to S180, S81 to S181, S82 to S182, S83 to S183, S84 to S184, U2 to U1, U1 to U2
Connections:
- C2 pad 1: /VBAT -> /VBUS
- J3 pad 1: +3V3 -> GND
- J3 pad 2: Net-(J3-Pad2) -> /SWDIO
- J3 pad 3: GND -> /SWDCLK
- J3 pad 4: Net-(J3-Pad4) -> +3V3
- J3 pad 6: Net-(J3-Pad6) -> /VBAT
- J3 pad 7: Net-(J3-Pad7) -> GND
- J3 pad 9: GND -> Net-(J3-Pad9)
- J4 pad 1: GND -> +3V3
- J4 pad 2: /SWDIO -> /SWDCLK
- J4 pad 3: /SWDCLK -> GND
- J4 pad 4: +3V3 -> /SWDIO
- J4 pad 6: /VBAT -> /SWO
- J4 pad 7: GND -> Net-(J4-Pad7)
- U2 pad 24: Net-(U1-Pad24) -> /USB_D+
- U2 pad 25: Net-(U1-Pad25) -> /USB_D-
- U2 pad 33: Net-(U1-Pad33) -> /USB_PU_CTRL
- U2 pad 34: Net-(U1-Pad34) -> /col4
- U2 pad 35: /col4 -> /col3
- U2 pad 36: /col3 -> /col2
- U2 pad 37: /col2 -> /col1
- U2 pad 38: /col1 -> Net-(U2-Pad38)
Routing:
- net GND: track 0.00 -> 287.8 mm, vias 0 -> 20
- net /USB_D-: track 0.00 -> 149.1 mm
- net /USB_D+: track 0.00 -> 148.1 mm
- net /VBUS: track 0.00 -> 8.09 mm, vias 0 -> 10
- net Net-(R4-Pad2): track 0.00 -> 4.71 mm
- net Net-(Q1-Pad3): track 0.00 -> 1.87 mm
- net /USB_PU_CTRL: track 0.00 -> 1.61 mm
- net +3V3: track 0.00 -> 1.61 mm
- net Net-(R3-Pad1): track 0.00 -> 1.60 mm
- net /VBAT: vias 0 -> 10
Other:
- rule trace_min: 0.2 -> 0.2032
- board text added: "3V3"
- board text added: "BAT"
- board text added: "CLK"
- board text added: "DIO"
- board text added: "GND"
- board text added: "SWD"

Commit message: finally completed?
Parts:
- removed D1: D, Diode_SMD:D_0805_2012Metric
- removed Q2: PMOS, Package_TO_SOT_SMD:SOT-23
- added C6: C, Capacitor_SMD:C_0603_1608Metric, B.Cu at (145.5, 136.7)
- added J4: Conn_01x10, Connector_PinHeader_2.54mm:PinHeader_1x10_P2.54mm_Vertical, F.Cu at (214.6, 156.2)
- added LED101: LED, LED_SMD:LED_0805_2012Metric, F.Cu at (64.8, 111.8)
- added Y1: 32.768Hz, Crystal:Crystal_DS26_D2.0mm_L6.0mm_Horizontal_1EP_style1, B.Cu at (142.0, 135.9)
- C1: value 1uF -> C
- J3: value Conn_01x10 -> JST_PH; footprint Connector_PinHeader_2.54mm:PinHeader_1x10_P2.54mm_Vertical -> Connector_JST:JST_PH_S2B-PH-K_1x02_P2.00mm_Horizontal; moved to B.Cu
- Q1: value PMOS -> Q_NMOS_DSG
- R1: value 10k -> R; footprint Resistor_SMD:R_0603_1608Metric -> Resistor_THT:R_Axial_DIN0207_L6.3mm_D2.5mm_P10.16mm_Horizontal
- R2: footprint Resistor_SMD:R_0603_1608Metric -> Capacitor_SMD:C_0603_1608Metric
- R5, R8: value R -> 10k
- R6, R7: value 10k -> 100k
- R9: value R -> 10k; footprint Resistor_THT:R_Axial_DIN0207_L6.3mm_D2.5mm_P10.16mm_Horizontal -> Resistor_SMD:R_0603_1608Metric; moved to B.Cu
- moved J3 125.9 mm to (101.6, 101.3), turned to 270 degrees
- moved C1 89.8 mm to (140.3, 136.7)
- moved R1 70.3 mm to (67.3, 134.8), turned to 270 degrees
- moved C5 67.6 mm to (160.3, 144.8), turned to 90 degrees
- moved Q1 65.4 mm to (88.9, 100.3), turned to 180 degrees
- moved U3 63.7 mm to (157.5, 144.8), turned to 0 degrees
- moved C4 59.3 mm to (154.7, 144.8), turned to 90 degrees
- moved R9 53.4 mm to (88.9, 102.9), turned to 0 degrees
- moved R2 47.3 mm to (146.6, 96.5)
- moved R8 23.5 mm to (96.0, 119.9)
- moved R5 21.6 mm to (87.6, 66.5), turned to 90 degrees
- moved D109 15.2 mm to (116.3, 140.5), turned to 90 degrees
- moved D106 15.0 mm to (107.7, 140.5), turned to 90 degrees
- moved D103 14.5 mm to (82.3, 140.5), turned to 90 degrees
- moved R10 13.5 mm to (64.8, 116.1), turned to 90 degrees
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- renumbered J4 to J5, LED103 to LED102, LED104 to LED103, LED101 to LED104, LED102 to LED105, LED105 to LED106, LED106 to LED107, LED107 to LED108, LED108 to LED109, LED109 to LED110, LED110 to LED111, LED111 to LED112, LED112 to LED113, LED113 to LED114, LED114 to LED115, LED115 to LED116, LED116 to LED117, LED117 to LED118, LED118 to LED119, LED119 to LED120, LED120 to LED121, LED121 to LED122, LED122 to LED123, LED123 to LED124, LED124 to LED125, LED125 to LED126, LED126 to LED127, LED127 to LED128, LED128 to LED129, LED129 to LED130, LED130 to LED131, LED131 to LED132, LED132 to LED133, LED133 to LED134, LED134 to LED135, LED135 to LED136, LED136 to LED137, LED137 to LED138, LED138 to LED139, LED139 to LED140, LED140 to LED141, LED141 to LED142, LED142 to LED143, LED143 to LED144, LED144 to LED145, LED145 to LED146, LED146 to LED147, LED147 to LED148, LED148 to LED149, LED149 to LED150, LED150 to LED151, LED151 to LED152, LED152 to LED153, LED153 to LED154, LED154 to LED155, LED155 to LED156, LED156 to LED157, LED157 to LED158, LED158 to LED159, LED159 to LED160, LED160 to LED161, LED161 to LED162, LED162 to LED163, LED163 to LED164, LED164 to LED165, LED165 to LED166, LED166 to LED167, LED167 to LED168, LED168 to LED169, LED169 to LED170, LED170 to LED171, LED171 to LED172, LED172 to LED173, LED173 to LED174, LED174 to LED175, LED175 to LED176, LED176 to LED177, LED177 to LED178, LED178 to LED179, LED179 to LED180, LED180 to LED181, LED181 to LED182, LED182 to LED183, LED183 to LED184, LED184 to LED185
Connections:
- C1 pad 1: /VBUS -> Net-(C1-Pad1)
- J3 pad 2: /SWDIO -> /VBAT
- LED102 pad 2: GND -> /Leds/LED-
- LED103 pad 2: GND -> /Leds/LED-
- LED104 pad 1: /Leds/CAPS_LED+ -> /Leds/LED+
- LED104 pad 2: /CAPS_LED -> /Leds/LED-
- LED105 pad 1: /Leds/CAPS_LED+ -> /Leds/LED+
- LED105 pad 2: /CAPS_LED -> /Leds/LED-
- LED106 pad 2: GND -> /Leds/LED-
- LED107 pad 2: GND -> /Leds/LED-
- LED108 pad 2: GND -> /Leds/LED-
- LED109 pad 1: GND -> /Leds/LED-
- LED110 pad 2: GND -> /Leds/LED-
- LED111 pad 2: GND -> /Leds/LED-
- LED112 pad 2: GND -> /Leds/LED-
- LED113 pad 2: GND -> /Leds/LED-
- LED114 pad 2: GND -> /Leds/LED-
- LED115 pad 1: GND -> /Leds/LED-
- LED116 pad 1: GND -> /Leds/LED-
- LED117 pad 2: GND -> /Leds/LED-
- LED118 pad 2: GND -> /Leds/LED-
- LED119 pad 2: GND -> /Leds/LED-
- LED120 pad 2: GND -> /Leds/LED-
- LED121 pad 2: GND -> /Leds/LED-
- LED122 pad 1: GND -> /Leds/LED-
- LED123 pad 2: GND -> /Leds/LED-
- LED124 pad 2: GND -> /Leds/LED-
- LED125 pad 2: GND -> /Leds/LED-
- LED126 pad 2: GND -> /Leds/LED-
- LED127 pad 2: GND -> /Leds/LED-
- LED128 pad 2: GND -> /Leds/LED-
- LED129 pad 2: GND -> /Leds/LED-
- LED130 pad 2: GND -> /Leds/LED-
- LED131 pad 2: GND -> /Leds/LED-
- LED132 pad 2: GND -> /Leds/LED-
- LED133 pad 2: GND -> /Leds/LED-
- LED134 pad 2: GND -> /Leds/LED-
- LED135 pad 2: GND -> /Leds/LED-
- LED136 pad 2: GND -> /Leds/LED-
- LED137 pad 2: GND -> /Leds/LED-
- LED138 pad 2: GND -> /Leds/LED-
- LED139 pad 2: GND -> /Leds/LED-
- LED140 pad 2: GND -> /Leds/LED-
- LED141 pad 2: GND -> /Leds/LED-
- LED142 pad 2: GND -> /Leds/LED-
- LED143 pad 2: GND -> /Leds/LED-
- LED144 pad 2: GND -> /Leds/LED-
- LED145 pad 2: GND -> /Leds/LED-
- LED146 pad 2: GND -> /Leds/LED-
- LED147 pad 2: GND -> /Leds/LED-
- LED148 pad 2: GND -> /Leds/LED-
- LED149 pad 2: GND -> /Leds/LED-
- LED150 pad 2: GND -> /Leds/LED-
- LED151 pad 2: GND -> /Leds/LED-
- LED152 pad 2: GND -> /Leds/LED-
- LED153 pad 2: GND -> /Leds/LED-
- LED154 pad 2: GND -> /Leds/LED-
- LED155 pad 2: GND -> /Leds/LED-
- LED156 pad 2: GND -> /Leds/LED-
- LED157 pad 2: GND -> /Leds/LED-
- LED158 pad 2: GND -> /Leds/LED-
- LED159 pad 1: GND -> /Leds/LED-
- LED160 pad 2: GND -> /Leds/LED-
- LED161 pad 2: GND -> /Leds/LED-
- LED162 pad 2: GND -> /Leds/LED-
- LED163 pad 2: GND -> /Leds/LED-
- LED164 pad 1: GND -> /Leds/LED-
- LED165 pad 1: GND -> /Leds/LED-
- LED166 pad 2: GND -> /Leds/LED-
- LED167 pad 2: GND -> /Leds/LED-
- LED168 pad 2: GND -> /Leds/LED-
- LED169 pad 2: GND -> /Leds/LED-
- LED170 pad 2: GND -> /Leds/LED-
- LED171 pad 2: GND -> /Leds/LED-
- LED172 pad 2: GND -> /Leds/LED-
- LED173 pad 1: GND -> /Leds/LED-
- LED174 pad 2: GND -> /Leds/LED-
- LED175 pad 2: GND -> /Leds/LED-
- LED176 pad 2: GND -> /Leds/LED-
- LED177 pad 2: GND -> /Leds/LED-
- LED178 pad 2: GND -> /Leds/LED-
- LED179 pad 2: GND -> /Leds/LED-
- LED180 pad 2: GND -> /Leds/LED-
- LED181 pad 2: GND -> /Leds/LED-
- LED182 pad 2: GND -> /Leds/LED-
- LED183 pad 2: GND -> /Leds/LED-
- LED184 pad 1: GND -> /Leds/LED-
- LED185 pad 2: GND -> /Leds/LED-
- Q1 pad 1: /USB_PU_CTRL -> /Leds/LED-
- Q1 pad 2: +3V3 -> GND
- Q1 pad 3: Net-(Q1-Pad3) -> /BKLT_LED
- R1 pad 2: /USB_PU_CTRL -> /Leds/LED+
- R2 pad 1: Net-(Q1-Pad3) -> /USB_D-
- R2 pad 2: /USB_D- -> /USB_PU
- R8 pad 1: +3V3 -> Net-(R8-Pad1)
- R8 pad 2: /BKLT_LED -> GND
- R9 pad 1: Net-(Q2-Pad3) -> /BKLT_LED
- R9 pad 2: /Leds/LED+ -> GND
- S109 pad 2: Net-(D104-Pad2) -> Net-(D104-Pad1)
- S110 pad 2: Net-(D104-Pad1) -> Net-(D104-Pad2)
- S116 pad 2: Net-(D107-Pad2) -> Net-(D107-Pad1)
- S117 pad 2: Net-(D107-Pad1) -> Net-(D107-Pad2)
- S122 pad 2: Net-(D110-Pad2) -> Net-(D110-Pad1)
- S123 pad 2: Net-(D110-Pad1) -> Net-(D110-Pad2)
- S130 pad 2: Net-(D114-Pad2) -> Net-(D114-Pad1)
- S131 pad 2: Net-(D114-Pad1) -> Net-(D114-Pad2)
- S135 pad 1: /row5 -> Net-(D116-Pad2)
- S135 pad 2: Net-(D116-Pad2) -> /row5
- S137 pad 2: Net-(D117-Pad2) -> Net-(D117-Pad1)
- S138 pad 2: Net-(D117-Pad1) -> Net-(D117-Pad2)
- S141 pad 2: Net-(D119-Pad2) -> Net-(D119-Pad1)
- S142 pad 2: Net-(D119-Pad1) -> Net-(D119-Pad2)
- S145 pad 2: Net-(D121-Pad2) -> Net-(D121-Pad1)
- S146 pad 2: Net-(D121-Pad1) -> Net-(D121-Pad2)
- S149 pad 2: Net-(D123-Pad2) -> Net-(D123-Pad1)
- S150 pad 2: Net-(D123-Pad1) -> Net-(D123-Pad2)
- S154 pad 2: Net-(D126-Pad2) -> Net-(D126-Pad1)
- S155 pad 2: Net-(D126-Pad1) -> Net-(D126-Pad2)
- S160 pad 2: Net-(D129-Pad2) -> Net-(D129-Pad1)
- S161 pad 2: Net-(D129-Pad1) -> Net-(D129-Pad2)
- S167 pad 2: Net-(D132-Pad2) -> Net-(D132-Pad1)
- S168 pad 2: Net-(D132-Pad1) -> Net-(D132-Pad2)
- S169 pad 2: Net-(D133-Pad1) -> Net-(D133-Pad2)
- S170 pad 1: /row4 -> Net-(D133-Pad1)
- S170 pad 2: Net-(D133-Pad2) -> /row4
- S171 pad 1: /row4 -> Net-(D133-Pad1)
- S171 pad 2: Net-(D133-Pad2) -> /row4
- S174 pad 2: Net-(D135-Pad2) -> Net-(D135-Pad1)
- S175 pad 2: Net-(D135-Pad2) -> Net-(D135-Pad1)
- S176 pad 2: Net-(D135-Pad1) -> Net-(D135-Pad2)
- S181 pad 1: Net-(D136-Pad1) -> /row4
- S181 pad 2: /row4 -> Net-(D136-Pad1)
- SW1 pad 1: /VBAT_SW -> /VBAT
- SW1 pad 2: /VBAT -> /VBAT_SW
- SW1 pad 3: Net-(SW1-Pad3) -> Net-(R8-Pad1)
- U2 pad 10: Net-(U2-Pad10) -> /col10
- U2 pad 11: Net-(U2-Pad11) -> /col9
- U2 pad 12: Net-(U2-Pad12) -> /col14
- U2 pad 13: Net-(U2-Pad13) -> /col13
- U2 pad 14: Net-(U2-Pad14) -> /col12
- U2 pad 15: Net-(U2-Pad15) -> /col11
- U2 pad 17: Net-(U2-Pad17) -> /row3
- U2 pad 18: Net-(U2-Pad18) -> /row2
- U2 pad 19: Net-(U2-Pad19) -> /row1
- U2 pad 2: Net-(U2-Pad2) -> /usr1
- U2 pad 20: Net-(U2-Pad20) -> /row4
- U2 pad 21: Net-(U2-Pad21) -> /col5
- U2 pad 22: Net-(U2-Pad22) -> /USB_D+
- U2 pad 23: Net-(U2-Pad23) -> /USB_D-
- U2 pad 24: /USB_D+ -> Net-(C6-Pad1)
- U2 pad 25: /USB_D- -> Net-(C1-Pad1)
- U2 pad 28: Net-(U2-Pad28) -> /CAPS_LED
- U2 pad 29: Net-(U2-Pad29) -> /BKLT_LED
- U2 pad 3: Net-(U2-Pad3) -> /usr2
- U2 pad 30: Net-(U2-Pad30) -> /col7
- U2 pad 31: Net-(U2-Pad31) -> /col8
- U2 pad 32: /VBAT_SENSE -> /USB_PU
- U2 pad 33: /USB_PU_CTRL -> /VBAT_SENSE
- U2 pad 4: Net-(U2-Pad4) -> /usr3
- U2 pad 7: Net-(U2-Pad7) -> /row5
- U2 pad 8: Net-(U2-Pad8) -> /col6
- U3 pad 4: Net-(U3-Pad4) -> GND
Routing:
- net /Leds/LED+: track 0.00 -> 1446.9 mm, vias 0 -> 12
- net /Leds/LED-: track 0.00 -> 1429.4 mm, vias 0 -> 11
- net /row5: track 0.00 -> 544.6 mm, vias 0 -> 6
- net /row1: track 0.00 -> 333.1 mm
- net /row3: track 0.00 -> 322.0 mm
- net /row2: track 0.00 -> 313.8 mm
- net /row4: track 0.00 -> 282.2 mm
- net /NCHG: track 0.00 -> 275.4 mm, vias 0 -> 4
- net /VBUS: track 8.09 -> 268.8 mm, vias 10 -> 2
- net +3V3: track 1.61 -> 236.5 mm, vias 0 -> 5
- net /col10: track 0.00 -> 229.5 mm, vias 0 -> 6
- net /VBAT: track 0.00 -> 228.1 mm, vias 10 -> 1
- net /col14: track 0.00 -> 219.3 mm, vias 0 -> 2
- net /col13: track 0.00 -> 202.4 mm, vias 0 -> 2
- net /col12: track 0.00 -> 185.4 mm, vias 0 -> 2
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- added copper zone on F.Cu, net (none)
- removed copper zone on B.Cu, net /VBAT
- removed copper zone on F.Cu, net /VBAT
- removed copper zone on B.Cu, net /VBUS
- removed copper zone on F.Cu, net /VBUS
Other:
- board text added: "5V"

Commit message: WIP
Parts:
- moved D116 3.30 mm to (181.1, 140.5)
- moved D105 1.02 mm to (103.9, 121.4), turned to 270 degrees
- renumbered C6 to C2, C2 to C3, C3 to C4, C4 to C5, C5 to C6, J5 to J4, J4 to J5, R10 to R1, R7 to R10, R1 to R3, R9 to R4, R3 to R5, R4 to R6, R5 to R7, R6 to R9
Connections:
- net /usr1 renamed /usr24
- net /usr2 renamed /usr23
- net /usr3 renamed /usr22
Routing:
- net Net-(D116-Pad2): track 27.6 -> 31.2 mm
- net /col14: track 219.3 -> 222.7 mm
- net /NCHG: track 275.4 -> 278.8 mm
- net +3V3: track 236.5 -> 233.5 mm, vias 5 -> 6
- net /col6: track 89.1 -> 86.2 mm
- net /col2: track 133.5 -> 135.5 mm
- net /SWO: track 54.0 -> 52.5 mm
- net /row1: track 333.1 -> 334.5 mm
- net /col10: track 229.5 -> 228.3 mm
- net Net-(D105-Pad1): track 22.9 -> 24.1 mm
- net /row2: track 313.8 -> 314.3 mm
- net GND: vias 67 -> 60
- removed copper zone on F.Cu, net (none)

Commit message: WIP
Parts:
- J5: footprint Connector_PinHeader_2.54mm:PinHeader_1x10_P2.54mm_Vertical -> header:PinHeader_1x10_P2.54mm_Vertical
Other:
- board text added: "22"
- board text added: "23"
- board text added: "24"

Commit message: WIP
Parts:
- D101, D102, D104, D105, D107, D108, D110, D111, D112, D113, D114, D115, D117, D118, D119, D120, D121, D122, D123, D124, D126, D127, D129, D130, D132, D133, D135, D136: value D_x2_KCom_AAK -> BAS70-05
- D103, D106, D109, D116, D125, D128, D131, D134, D137: value D -> BAS70-05
- LED1, LED101: value LED -> Red_LED
- MXST1, MXST10, MXST11, MXST12, MXST13, MXST14, MXST15, MXST2, MXST3, MXST4, MXST5, MXST6, MXST7, MXST8, MXST9: value Stabilizer_Mounting -> Cherry_Stabilizer
- Q1: value Q_NMOS_DSG -> Q_NMOS_GSD
- R1, R5: value R -> 1.5k
- Y1: value 32.768Hz -> 32.768kHz
- moved R4 5.09 mm to (89.2, 97.8), turned to 180 degrees
Connections:
- Q1 pad 1: /Leds/LED- -> /BKLT_LED
- Q1 pad 3: /BKLT_LED -> /Leds/LED-
Routing:
- net /Leds/LED-: track 1429.4 -> 1431.7 mm
- net /BKLT_LED: track 114.5 -> 112.6 mm
- net GND: track 190.7 -> 189.3 mm, vias 60 -> 59
- net /CAPS_LED: track 143.9 -> 144.7 mm
Other:
- board text added: "SWDIO"
- board text removed: "DIO"

Commit message: almost ready
Parts:
- added TP1: TestPoint, header:PinHeader_1x04_P2.54mm_Vertical, F.Cu at (64.8, 88.9)
- Q1: value Q_NMOS_GSD -> Q_NMOS
Connections:
- J1 pad 4: Net-(J1-Pad4) -> (no net)
- J4 pad 10: Net-(J4-Pad10) -> (no net)
- J4 pad 7: Net-(J4-Pad7) -> (no net)
- J4 pad 8: Net-(J4-Pad8) -> (no net)
- U2 pad 38: Net-(U2-Pad38) -> (no net)
- U3 pad 4: GND -> (no net)
Routing:
- net /USB_D-: track 154.4 -> 179.6 mm
- net /USB_D+: track 153.2 -> 178.3 mm
- net Net-(D101-Pad2): track 20.7 -> 18.1 mm
- net /Leds/LED+: track 1447.2 -> 1448.7 mm, vias 12 -> 13
- net /SWDCLK: track 58.0 -> 59.1 mm
- net /NCHG: track 278.8 -> 277.9 mm
- net /SWO: track 52.5 -> 51.9 mm
- net /Leds/LED-: track 1431.7 -> 1432.2 mm, vias 11 -> 12
