File: keyboard.sch (KiCad schematic (older format))
At the start: 18 parts, among them J1 USB_B_Micro, J2 JST_PH, SW1 SW_Push, U1 BL652

Commit message: WIP
Parts:
- removed JP?: Jumper_3_Bridged12, symbol Jumper:Jumper_3_Bridged12
- removed Q?: Q_NMOS_DSG, symbol Device:Q_NMOS_DSG
- removed R? (x2): R, symbol Device:R
- removed U?: BQ21040, symbol batmgmt:BQ21040
- added C1: 1uF, Capacitor_SMD:C_0603_1608Metric, symbol Device:C
- added D1: D, Diode_SMD:D_0805_2012Metric, symbol Device:D
- added J3: Conn_01x08, Connector_PinHeader_2.54mm:PinHeader_1x08_P2.54mm_Vertical, symbol Connector_Generic:Conn_01x08
- added J4: Conn_ARM_JTAG_SWD_10, swd:PinHeader_2x05_P1.27mm_Vertical_SMD, symbol Connector:Conn_ARM_JTAG_SWD_10
- added Q1, Q2: PMOS, Package_TO_SOT_SMD:SOT-23, symbol Device:Q_PMOS_GSD
- added R1, R6, R7: 10k, Resistor_SMD:R_0603_1608Metric, symbol Device:R
- added R10, R9: R, Resistor_THT:R_Axial_DIN0207_L6.3mm_D2.5mm_P10.16mm_Horizontal, symbol Device:R
- added R2: 1.5k, Resistor_SMD:R_0603_1608Metric, symbol Device:R
- added R8: R, Resistor_SMD:R_0603_1608Metric, symbol Device:R
- added SW1: SSSS912000, switch:SSSS912000, symbol Switch:SW_SPDT
- added U1: BQ21040, Package_TO_SOT_SMD:SOT-23-6, symbol batmgmt:BQ21040
- C2, C3: renamed from C?; footprint (none) -> Capacitor_SMD:C_0603_1608Metric
- C4, C5: renamed from C?; value C -> 1uF; footprint (none) -> Capacitor_SMD:C_0603_1608Metric
- J2: footprint Connector_JST:JST_PH_S2B-PH-SM4-TB_1x02-1MP_P2.00mm_Horizontal -> Connector_JST:JST_PH_S2B-PH-K_1x02_P2.00mm_Horizontal
- LED1: renamed from D?; footprint (none) -> LED_SMD:LED_0805_2012Metric
- R3, R4, R5: renamed from R?; footprint (none) -> Resistor_SMD:R_0603_1608Metric
- U3: renamed from U?; value TLV70033_SOT23-5 -> TLV70033
- renumbered SW1 to SW2, U1 to U2
Connections:
- net labels added: BKLT_LED, SWDCLK, SWDIO, USB_PU_CTRL, VBAT_SENSE, VBAT_SW
- net labels removed: LED_PWM, V_UNREG
- wire segments 60 -> 93
- no-connect marks 3 -> 7
Other:
- note added: "Battery connector"
- note added: "Charging indicator"
- note added: "Optional charger bypass\nOnly use when operating without a battery"
- note removed: "battery connector"

Commit message: WIP
Parts:
- removed SW2: SW_Push, dtsm:KSEM31GLFS, symbol Switch:SW_Push
- J3: value Conn_01x08 -> Conn_01x10; footprint Connector_PinHeader_2.54mm:PinHeader_1x08_P2.54mm_Vertical -> Connector_PinHeader_2.54mm:PinHeader_1x10_P2.54mm_Vertical; symbol Connector_Generic:Conn_01x08 -> Connector_Generic:Conn_01x10
- R10: footprint Resistor_THT:R_Axial_DIN0207_L6.3mm_D2.5mm_P10.16mm_Horizontal -> Resistor_SMD:R_0603_1608Metric
Connections:
- wire segments 93 -> 106
- no-connect marks 7 -> 5
Changed lines of the file:
@@
 $EndSheet
-$Comp
-L Switch:SW_Push SW2
-U 1 1 5B911142
-P 15250 3600
-F 0 "SW2" H 15250 3885 50  0000 C CNN
-F 1 "SW_Push" H 15250 3794 50  0000 C CNN
-F 2 "dtsm:KSEM31GLFS" H 15250 3800 50  0001 C CNN
-F 3 "" H 15250 3800 50  0001 C CNN
-	1    15250 3600
-	1    0    0    -1
-$EndComp
 $Comp
 L Connector:USB_B_Micro J1
@@
 	4700 2100 4400 2100
 Wire Wire Line
-	6900 6100 7400 6100
-Text Label 6950 6100 0    60   ~ 0
+	6900 6000 7400 6000
+Text Label 6950 6000 0    60   ~ 0
 col1
-Text Label 6950 6000 0    60   ~ 0
+Text Label 6950 5900 0    60   ~ 0
 col2
 Wire Wire Line
-	6900 6000 7400 6000
-Wire Wire Line
 	6900 5900 7400 5900
-Text Label 6950 5900 0    60   ~ 0
+Wire Wire Line
+	6900 5800 7400 5800
+Text Label 6950 5800 0    60   ~ 0
 col3
 NoConn ~ 1400 2100
-Text Label 6950 5800 0    60   ~ 0
+Text Label 6950 5700 0    60   ~ 0
 col4
 Wire Wire Line
-	6900 5800 7400 5800
+	6900 5700 7400 5700
 Text Label 6950 5100 0    60   ~ 0
 SWDCLK
@@
 Text Label 11050 3500 0    60   ~ 0
 CAPS_LED
-NoConn ~ 15050 3600
-NoConn ~ 15450 3600
 NoConn ~ 5800 2150
 Text Label 5850 1950 0    60   ~ 0
@@
 Text Label 1600 2950 3    50   ~ 0
 USB_PU_CTRL
-Wire Wire Line
-	1600 2900 1600 3600
 $Comp
 L Device:R R1
@@
 Connection ~ 2250 3400
 Wire Wire Line
-	2250 3400 2250 3850
-Wire Wire Line
 	2250 1800 2250 3400
 $Comp
@@
 F 0 "R10" H 11800 3200 50  0000 L CNN
 F 1 "R" H 11800 3100 50  0000 L CNN
-F 2 "Resistor_THT:R_Axial_DIN0207_L6.3mm_D2.5mm_P10.16mm_Horizontal" V 11680 3150 50  0001 C CNN
+F 2 "Resistor_SMD:R_0603_1608Metric" V 11680 3150 50  0001 C CNN
 F 3 "~" H 11750 3150 50  0001 C CNN
 	1    11750 3150
@@
 	11050 3500 11050 3850
 $Comp
-L Connector_Generic:Conn_01x08 J3
+L Connector_Generic:Conn_01x10 J3
 U 1 1 5B6D3C72
 P 10650 7150
 F 0 "J3" H 10730 7142 50  0000 L CNN
-F 1 "Conn_01x08" H 10730 7051 50  0000 L CNN
-F 2 "Connector_PinHeader_2.54mm:PinHeader_1x08_P2.54mm_Vertical" H 10650 7150 50  0001 C CNN
+F 1 "Conn_01x10" H 10730 7051 50  0000 L CNN
+F 2 "Connector_PinHeader_2.54mm:PinHeader_1x10_P2.54mm_Vertical" H 10650 7150 50  0001 C CNN
 F 3 "~" H 10650 7150 50  0001 C CNN
 	1    10650 7150
 	1    0    0    -1
 $EndComp
+Text Label 10350 6850 2    60   ~ 0
+SWDIO
 Text Label 10350 6950 2    60   ~ 0
-SWDIO
-Text Label 10350 7050 2    60   ~ 0
 SWDCLK
 $Comp
 L power:+3.3V #PWR013
 U 1 1 5B6DEDDE
+P 10450 7050
+F 0 "#PWR013" H 10450 6900 50  0001 C CNN
+F 1 "+3.3V" V 10450 7150 60  0000 L TNN
+F 2 "" H 10450 7050 50  0001 C CNN
+F 3 "" H 10450 7050 50  0001 C CNN
+	1    10450 7050
+	0    -1   -1   0
+$EndComp
+$Comp
+L power:GND #PWR014
+U 1 1 5B6DEF09
 P 10450 7150
-F 0 "#PWR013" H 10450 7000 50  0001 C CNN
-F 1 "+3.3V" V 10450 7250 60  0000 L TNN
+F 0 "#PWR014" H 10450 6900 50  0001 C CNN
+F 1 "GND" V 10450 7050 60  0000 R BNN
 F 2 "" H 10450 7150 50  0001 C CNN
 F 3 "" H 10450 7150 50  0001 C CNN
 	1    10450 7150
-	0    -1   -1   0
-$EndComp
-$Comp
-L power:GND #PWR014
-U 1 1 5B6DEF09
-P 10450 7250
-F 0 "#PWR014" H 10450 7000 50  0001 C CNN
-F 1 "GND" V 10450 7150 60  0000 R BNN
-F 2 "" H 10450 7250 50  0001 C CNN
-F 3 "" H 10450 7250 50  0001 C CNN
-	1    10450 7250
 	0    1    1    0
 $EndComp
@@
 L power:GND #PWR012
 U 1 1 5B6E8E96
-P 10450 6850
-F 0 "#PWR012" H 10450 6600 50  0001 C CNN
-F 1 "GND" V 10450 6750 60  0000 R BNN
-F 2 "" H 10450 6850 50  0001 C CNN
-F 3 "" H 10450 6850 50  0001 C CNN
-	1    10450 6850
+P 10450 6750
+F 0 "#PWR012" H 10450 6500 50  0001 C CNN
+F 1 "GND" V 10450 6650 60  0000 R BNN
+F 2 "" H 10450 6750 50  0001 C CNN
+F 3 "" H 10450 6750 50  0001 C CNN
+	1    10450 6750
 	0    1    1    0
 $EndComp
 Wire Wire Line
-	10450 7050 10350 7050
-Wire Wire Line
-	10350 6950 10450 6950
+	10450 6950 10350 6950
+Wire Wire Line
+	10350 6850 10450 6850
 $Comp
 L power:GND #PWR015
 U 1 1 5B6F06B3
-P 10450 7450
-F 0 "#PWR015" H 10450 7200 50  0001 C CNN
-F 1 "GND" V 10450 7350 60  0000 R BNN
-F 2 "" H 10450 7450 50  0001 C CNN
-F 3 "" H 10450 7450 50  0001 C CNN
-	1    10450 7450
+P 10450 7350
+F 0 "#PWR015" H 10450 7100 50  0001 C CNN
+F 1 "GND" V 10450 7250 60  0000 R BNN
+F 2 "" H 10450 7350 50  0001 C CNN
+F 3 "" H 10450 7350 50  0001 C CNN
+	1    10450 7350
 	0    1    1    0
 $EndComp
 Text Label 6150 1500 2    60   ~ 0
 VBAT
-Text Label 10350 7350 2    60   ~ 0
+Text Label 10350 7250 2    60   ~ 0
 VBAT
 Wire Wire Line
-	10450 7350 10350 7350
+	10450 7250 10350 7250
 Connection ~ 5000 1500
 $Comp
@@
 Wire Wire Line
 	7900 5500 6900 5500
+Text Label 10150 5300 2    60   ~ 0
+SWDIO
+Text Label 10150 5400 2    60   ~ 0
+SWDCLK
+Wire Wire Line
+	10200 5400 10100 5400
+Text Label 10150 5500 2    60   ~ 0
+SWO
+Wire Wire Line
+	10200 5500 10100 5500
+Wire Wire Line
+	10100 5300 10200 5300
+Wire Wire Line
+	4300 3850 2300 3850
+Wire Wire Line
+	2250 3900 4250 3900
+Wire Wire Line
+	4250 3900 4250 5100
+Wire Wire Line
+	2250 3400 2250 3900
+Wire Wire Line
+	6900 5600 8350 5600
+Wire Wire Line
+	8350 5600 8350 3950
+Wire Wire Line
+	8350 3950 1600 3950
+Wire Wire Line
+	1600 2900 1600 3950
+Wire Wire Line
+	4900 5200 4300 5200
+Wire Wire Line
+	4300 3850 4300 5100
+Wire Wire Line
+	4300 5100 4300 5200
+Wire Wire Line
+	4250 5100 4900 5100
 Wire Bus Line
 	2150 5250 2150 7850

Commit message: finally completed?
Parts:
- removed D1: D, Diode_SMD:D_0805_2012Metric, symbol Device:D
- removed Q1, Q2: PMOS, Package_TO_SOT_SMD:SOT-23, symbol Device:Q_PMOS_GSD
- added C6: C, Capacitor_SMD:C_0603_1608Metric, symbol Device:C
- added J3: JST_PH, Connector_JST:JST_PH_S2B-PH-K_1x02_P2.00mm_Horizontal, symbol Connector_Generic:Conn_01x02
- added Q1: Q_NMOS_DSG, Package_TO_SOT_SMD:SOT-23, symbol Device:Q_NMOS_DSG
- added Y1: 32.768Hz, Crystal:Crystal_DS26_D2.0mm_L6.0mm_Horizontal_1EP_style1, symbol Device:Crystal
- C1: value 1uF -> C
- R1: value 10k -> R; footprint Resistor_SMD:R_0603_1608Metric -> Resistor_THT:R_Axial_DIN0207_L6.3mm_D2.5mm_P10.16mm_Horizontal
- R2: footprint Resistor_SMD:R_0603_1608Metric -> Capacitor_SMD:C_0603_1608Metric
- R5, R8: value R -> 10k
- R6, R7: value 10k -> 100k
- R9: value R -> 10k; footprint Resistor_THT:R_Axial_DIN0207_L6.3mm_D2.5mm_P10.16mm_Horizontal -> Resistor_SMD:R_0603_1608Metric
- U3: symbol Regulator_Linear:TLV70033_SOT23-5 -> vreg:TLV70033_SOT23-5
- renumbered J3 to J4, J4 to J5
Connections:
- net labels added: USB_PU, usr1, usr2, usr3
- net labels removed: USB_PU_CTRL
- wire segments 106 -> 133
Other:
- note added: "100mA max led current"
- note added: "Battery connectors\nPopulate only one"
- note added: "When operating without battery,\nshort VBUS and VBAT to bypass charger"
- note removed: "Battery connector"
- note removed: "Optional charger bypass\nOnly use when operating without a battery"

Commit message: WIP
Parts:
- renumbered C6 to C2, C2 to C3, C3 to C4, C4 to C5, C5 to C6, J5 to J4, J4 to J5, R10 to R1, R7 to R10, R1 to R3, R9 to R4, R3 to R5, R4 to R6, R5 to R7, R6 to R9
Connections:
- net labels added: usr22, usr23, usr24
- net labels removed: usr1, usr2, usr3
- wire segments 133 -> 140

Commit message: WIP
Parts:
- J5: footprint Connector_PinHeader_2.54mm:PinHeader_1x10_P2.54mm_Vertical -> header:PinHeader_1x10_P2.54mm_Vertical
Changed lines of the file:
@@
 EESchema Schematic File Version 4
-LIBS:keyboard-cache
 EELAYER 26 0
 EELAYER END
@@
 F 0 "J5" H 10330 7442 50  0000 L CNN
 F 1 "Conn_01x10" H 10330 7351 50  0000 L CNN
-F 2 "Connector_PinHeader_2.54mm:PinHeader_1x10_P2.54mm_Vertical" H 10250 7450 50  0001 C CNN
+F 2 "header:PinHeader_1x10_P2.54mm_Vertical" H 10250 7450 50  0001 C CNN
 F 3 "~" H 10250 7450 50  0001 C CNN
 	1    10250 7450

Commit message: WIP
Parts:
- LED1: value LED -> Red_LED
- Q1: value Q_NMOS_DSG -> Q_NMOS_GSD; symbol Device:Q_NMOS_DSG -> Device:Q_NMOS_GSD
- R1, R5: value R -> 1.5k
- Y1: value 32.768Hz -> 32.768kHz
Changed lines of the file:
@@
 P 3500 1950
 F 0 "R5" H 3550 2000 50  0000 L CNN
-F 1 "R" H 3550 1900 50  0000 L CNN
+F 1 "1.5k" H 3550 1900 50  0000 L CNN
 F 2 "Resistor_SMD:R_0603_1608Metric" V 3430 1950 50  0001 C CNN
 F 3 "~" H 3500 1950 50  0001 C CNN
@@
 P 5000 2350
 F 0 "LED1" V 5000 2400 50  0000 L CNN
-F 1 "LED" V 5050 2300 50  0001 R CNN
+F 1 "Red_LED" V 5050 2300 50  0001 R CNN
 F 2 "LED_SMD:LED_0805_2012Metric" H 5000 2350 50  0001 C CNN
 F 3 "~" H 5000 2350 50  0001 C CNN
@@
 F 1 "SSSS912000" H 7150 1800 50  0001 C CNN
 F 2 "switch:SSSS912000" H 7150 1600 50  0001 C CNN
-F 3 "" H 7150 1600 50  0001 C CNN
+F 3 "https://www.alps.com/prod/info/E/HTML/Switch/Slide/SSSS9/SSSS912000.html" H 7150 1600 50  0001 C CNN
 	1    7150 1600
 	-1   0    0    -1
@@
 BKLT_LED
 $Comp
-L Device:Q_NMOS_DSG Q1
+L Device:Q_NMOS_GSD Q1
 U 1 1 5B62F2AA
 P 2100 9150
-F 0 "Q1" H 2305 9196 50  0000 L CNN
-F 1 "Q_NMOS_DSG" H 2305 9105 50  0000 L CNN
+F 0 "Q1" H 2300 9200 50  0000 L CNN
+F 1 "Q_NMOS_GSD" H 2300 9100 50  0000 L CNN
 F 2 "Package_TO_SOT_SMD:SOT-23" H 2300 9250 50  0001 C CNN
 F 3 "~" H 2100 9150 50  0001 C CNN
@@
 P 1950 8400
 F 0 "R1" H 2000 8450 50  0000 L CNN
-F 1 "R" H 2000 8350 50  0000 L CNN
+F 1 "1.5k" H 2000 8350 50  0000 L CNN
 F 2 "Resistor_SMD:R_0603_1608Metric" V 1880 8400 50  0001 C CNN
 F 3 "~" H 1950 8400 50  0001 C CNN
@@
 P 3400 5800
 F 0 "Y1" H 3400 6050 50  0000 C CNN
-F 1 "32.768Hz" H 3400 5950 50  0000 C CNN
+F 1 "32.768kHz" H 3400 5950 50  0000 C CNN
 F 2 "Crystal:Crystal_DS26_D2.0mm_L6.0mm_Horizontal_1EP_style1" H 3400 5800 50  0001 C CNN
 F 3 "~" H 3400 5800 50  0001 C CNN

Commit message: almost ready
Parts:
- Q1: value Q_NMOS_GSD -> Q_NMOS
Connections:
- wire segments 140 -> 138
- no-connect marks 5 -> 6
Changed lines of the file:
@@
 EESchema Schematic File Version 4
+LIBS:keyboard-cache
 EELAYER 26 0
 EELAYER END
@@
 encoding utf-8
 Sheet 1 4
-Title "ukbdc - schematic"
-Date "17 jul 2013"
+Title ""
+Date "2018-08-12"
 Rev ""
-Comp "komar"
+Comp ""
 Comment1 ""
 Comment2 ""
@@
 Wire Wire Line
 	2300 1700 2300 3850
-Text Label 2100 2900 2    50   ~ 0
+Text Label 2150 2900 2    60   ~ 0
 USB_PU
 $Comp
@@
 Wire Wire Line
 	9350 1600 9550 1600
-Wire Wire Line
-	9050 2000 9350 2000
-Wire Wire Line
-	9350 1700 9350 2000
-Connection ~ 9350 2000
-Wire Wire Line
-	9350 2000 9550 2000
 $Comp
 L Connector_Generic:Conn_01x02 J3
@@
 P 2100 9150
 F 0 "Q1" H 2300 9200 50  0000 L CNN
-F 1 "Q_NMOS_GSD" H 2300 9100 50  0000 L CNN
+F 1 "Q_NMOS" H 2300 9100 50  0000 L CNN
 F 2 "Package_TO_SOT_SMD:SOT-23" H 2300 9250 50  0001 C CNN
 F 3 "~" H 2100 9150 50  0001 C CNN
@@
 	2250 3200 2250 3900
 Wire Wire Line
-	1800 2900 1800 3950
-Wire Wire Line
 	1800 2900 2150 2900
 Wire Wire Line
-	1800 3950 7400 3950
-Wire Wire Line
 	6900 5100 7600 5100
 Wire Wire Line
 	6900 5200 7600 5200
-Wire Wire Line
-	7400 3950 7400 5500
 Wire Wire Line
 	7400 5500 6900 5500
@@
 Entry Wire Line
 	7600 6400 7700 6300
-Text Label 6950 5500 0    50   ~ 0
+Text Label 6950 5500 0    60   ~ 0
 USB_PU
 Text Label 6950 5600 0    60   ~ 0
@@
 Wire Wire Line
 	3750 5200 4900 5200
+Wire Wire Line
+	1800 4000 7400 4000
+Wire Wire Line
+	7400 4000 7400 5500
+Wire Wire Line
+	1800 2900 1800 4000
+Wire Wire Line
+	9050 2000 9550 2000
+NoConn ~ 9350 1700
 Wire Bus Line
 	7700 5000 7700 6750

Commit message: I think we are ready
Parts:
- J4: Part (none) -> FTSH-105-01-L-DV-K
- R2: footprint Capacitor_SMD:C_0603_1608Metric -> Resistor_SMD:R_0603_1608Metric
- R4: value 10k -> 100k
Changed lines of the file:
@@
 F 2 "swd:PinHeader_2x05_P1.27mm_Vertical_SMD" H 9950 4950 50  0001 L TNN
 F 3 "http://infocenter.arm.com/help/topic/com.arm.doc.faqs/attached/13634/cortex_debug_connectors.pdf" V 9550 4250 50  0001 C CNN
+F 4 "FTSH-105-01-L-DV-K" H 9900 5500 50  0001 C CNN "Part"
 	1    9900 5500
 	-1   0    0    -1
@@
 F 0 "R2" H 2200 3000 50  0000 L CNN
 F 1 "1.5k" H 2200 3100 50  0000 L CNN
-F 2 "Capacitor_SMD:C_0603_1608Metric" V 2080 3050 50  0001 C CNN
+F 2 "Resistor_SMD:R_0603_1608Metric" V 2080 3050 50  0001 C CNN
 F 3 "~" H 2150 3050 50  0001 C CNN
 	1    2150 3050
@@
 P 2300 9300
 F 0 "R4" H 2250 9350 50  0000 R CNN
-F 1 "10k" H 2250 9250 50  0000 R CNN
+F 1 "100k" H 2250 9250 50  0000 R CNN
 F 2 "Resistor_SMD:R_0603_1608Metric" V 2230 9300 50  0001 C CNN
 F 3 "~" H 2300 9300 50  0001 C CNN
