File: keyboard.sch (KiCad schematic (older format))
At the start: 28 parts, among them J1 USB_B_Micro, J2 JST_PH, J3 JST_PH, J4 Conn_ARM_JTAG_SWD_10, J5 Conn_01x10, Q1 Q_NMOS, SW1 SSSS912000, U1 BQ21040, U2 BL652, U3 TLV70033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

Commit message: Final touchups
Connections:
- wire segments 138 -> 139
- no-connect marks 6 -> 5
Changed lines of the file:
@@
 encoding utf-8
 Sheet 1 4
-Title ""
+Title "BLU60"
 Date "2018-08-12"
-Rev ""
+Rev "v0.1"
 Comp ""
 Comment1 ""
@@
 Text Label 6950 5800 0    60   ~ 0
 col3
-NoConn ~ 1400 2100
 Text Label 6950 5700 0    60   ~ 0
 col4
@@
 	9050 2000 9550 2000
 NoConn ~ 9350 1700
+Wire Wire Line
+	1400 2100 1500 2100
+Connection ~ 1500 2100
 Wire Bus Line
 	7700 5000 7700 6750

Commit message: Fixing up my stupid mistake
Changed lines of the file:
@@
 	1    0    0    -1
 $EndComp
+Text Label 9950 7150 2    60   ~ 0
+SWDIO
 Text Label 9950 7050 2    60   ~ 0
-SWDIO
-Text Label 9950 7150 2    60   ~ 0
 SWDCLK
 $Comp
@@
 Wire Wire Line
 	7950 1600 8550 1600
+Text Label 9350 5500 2    60   ~ 0
+SWDIO
 Text Label 9350 5400 2    60   ~ 0
-SWDIO
-Text Label 9350 5500 2    60   ~ 0
 SWDCLK
 Text Label 9350 5600 2    60   ~ 0
