File: leds.sch (KiCad schematic (older format))
At the start: 85 parts

Commit message: WIP
Parts:
- removed LED3: LED, mx1a:MX1A-led_no3d, symbol Device:LED
- LED101: renamed from LED1; symbol Device:LED -> led:LED_AK
- LED102: renamed from LED2; symbol Device:LED -> led:LED_AK
- LED103: renamed from LED4; symbol Device:LED -> led:LED_AK
- LED104: renamed from LED5; symbol Device:LED -> led:LED_AK
- LED105: renamed from LED6; symbol Device:LED -> led:LED_AK
- LED106: renamed from LED7; symbol Device:LED -> led:LED_AK
- LED107: renamed from LED8; symbol Device:LED -> led:LED_AK
- LED108: renamed from LED9; symbol Device:LED -> led:LED_KA
- LED109: renamed from LED10; symbol Device:LED -> led:LED_AK
- LED110: renamed from LED11; symbol Device:LED -> led:LED_AK
- LED111: renamed from LED12; symbol Device:LED -> led:LED_AK
- LED112: renamed from LED13; symbol Device:LED -> led:LED_AK
- LED113: renamed from LED14; symbol Device:LED -> led:LED_AK
- LED114: renamed from LED15; symbol Device:LED -> led:LED_KA
- LED115: renamed from LED16; symbol Device:LED -> led:LED_KA
- LED116: renamed from LED17; symbol Device:LED -> led:LED_AK
- LED117: renamed from LED18; symbol Device:LED -> led:LED_AK
- LED118: renamed from LED19; symbol Device:LED -> led:LED_AK
- LED119: renamed from LED20; symbol Device:LED -> led:LED_AK
- LED120: renamed from LED21; symbol Device:LED -> led:LED_AK
- LED121: renamed from LED22; symbol Device:LED -> led:LED_KA
- LED122: renamed from LED23; symbol Device:LED -> led:LED_AK
- LED123: renamed from LED24; symbol Device:LED -> led:LED_AK
- LED124: renamed from LED25; symbol Device:LED -> led:LED_AK
- LED125: renamed from LED26; symbol Device:LED -> led:LED_AK
- LED126: renamed from LED27; symbol Device:LED -> led:LED_AK
- LED127: renamed from LED28; symbol Device:LED -> led:LED_AK
- LED128: renamed from LED29; symbol Device:LED -> led:LED_AK
- LED129: renamed from LED30; symbol Device:LED -> led:LED_AK
- LED130: renamed from LED31; symbol Device:LED -> led:LED_AK
- LED131: renamed from LED32; symbol Device:LED -> led:LED_AK
- LED132: renamed from LED33; symbol Device:LED -> led:LED_AK
- LED133: renamed from LED34; symbol Device:LED -> led:LED_AK
- LED134: renamed from LED35; symbol Device:LED -> led:LED_AK
- LED135: renamed from LED36; symbol Device:LED -> led:LED_AK
- LED136: renamed from LED37; symbol Device:LED -> led:LED_AK
- LED137: renamed from LED38; symbol Device:LED -> led:LED_AK
- LED138: renamed from LED39; symbol Device:LED -> led:LED_AK
- LED139: renamed from LED40; symbol Device:LED -> led:LED_AK
- LED140: renamed from LED41; symbol Device:LED -> led:LED_AK
- LED141: renamed from LED42; symbol Device:LED -> led:LED_AK
- LED142: renamed from LED43; symbol Device:LED -> led:LED_AK
- LED143: renamed from LED44; symbol Device:LED -> led:LED_AK
- LED144: renamed from LED45; symbol Device:LED -> led:LED_AK
- LED145: renamed from LED46; symbol Device:LED -> led:LED_AK
- LED146: renamed from LED47; symbol Device:LED -> led:LED_AK
- LED147: renamed from LED48; symbol Device:LED -> led:LED_AK
- LED148: renamed from LED49; symbol Device:LED -> led:LED_AK
- LED149: renamed from LED50; symbol Device:LED -> led:LED_AK
- LED150: renamed from LED51; symbol Device:LED -> led:LED_AK
- LED151: renamed from LED52; symbol Device:LED -> led:LED_AK
- LED152: renamed from LED53; symbol Device:LED -> led:LED_AK
- LED153: renamed from LED54; symbol Device:LED -> led:LED_AK
- LED154: renamed from LED55; symbol Device:LED -> led:LED_AK
- LED155: renamed from LED56; symbol Device:LED -> led:LED_AK
- LED156: renamed from LED57; symbol Device:LED -> led:LED_AK
- LED157: renamed from LED58; symbol Device:LED -> led:LED_AK
- LED158: renamed from LED59; symbol Device:LED -> led:LED_KA
- LED159: renamed from LED60; symbol Device:LED -> led:LED_AK
- LED160: renamed from LED61; symbol Device:LED -> led:LED_AK
- LED161: renamed from LED62; symbol Device:LED -> led:LED_AK
- LED162: renamed from LED63; symbol Device:LED -> led:LED_AK
- LED163: renamed from LED64; symbol Device:LED -> led:LED_KA
- LED164: renamed from LED65; symbol Device:LED -> led:LED_KA
- LED165: renamed from LED66; symbol Device:LED -> led:LED_AK
- LED166: renamed from LED67; symbol Device:LED -> led:LED_AK
- LED167: renamed from LED68; symbol Device:LED -> led:LED_AK
- LED168: renamed from LED69; symbol Device:LED -> led:LED_AK
- LED169: renamed from LED70; symbol Device:LED -> led:LED_AK
- LED170: renamed from LED71; symbol Device:LED -> led:LED_AK
- LED171: renamed from LED72; symbol Device:LED -> led:LED_AK
- LED172: renamed from LED73; symbol Device:LED -> led:LED_KA
- LED173: renamed from LED74; symbol Device:LED -> led:LED_AK
- LED174: renamed from LED75; symbol Device:LED -> led:LED_AK
- LED175: renamed from LED76; symbol Device:LED -> led:LED_AK
- LED176: renamed from LED77; symbol Device:LED -> led:LED_AK
- LED177: renamed from LED78; symbol Device:LED -> led:LED_AK
- LED178: renamed from LED79; symbol Device:LED -> led:LED_AK
- LED179: renamed from LED80; symbol Device:LED -> led:LED_AK
- LED180: renamed from LED81; symbol Device:LED -> led:LED_AK
- LED181: renamed from LED82; symbol Device:LED -> led:LED_AK
- LED182: renamed from LED83; symbol Device:LED -> led:LED_AK
- LED183: renamed from LED84; symbol Device:LED -> led:LED_KA
- LED184: renamed from LED85; symbol Device:LED -> led:LED_AK
Connections:
- net labels added: CAPS_LED+
- wire segments 202 -> 201

Commit message: finally completed?
Parts:
- added LED101: LED, LED_SMD:LED_0805_2012Metric, symbol Device:LED
- renumbered LED103 to LED102, LED104 to LED103, LED101 to LED104, LED102 to LED105, LED105 to LED106, LED106 to LED107, LED107 to LED108, LED108 to LED109, LED109 to LED110, LED110 to LED111, LED111 to LED112, LED112 to LED113, LED113 to LED114, LED114 to LED115, LED115 to LED116, LED116 to LED117, LED117 to LED118, LED118 to LED119, LED119 to LED120, LED120 to LED121, LED121 to LED122, LED122 to LED123, LED123 to LED124, LED124 to LED125, LED125 to LED126, LED126 to LED127, LED127 to LED128, LED128 to LED129, LED129 to LED130, LED130 to LED131, LED131 to LED132, LED132 to LED133, LED133 to LED134, LED134 to LED135, LED135 to LED136, LED136 to LED137, LED137 to LED138, LED138 to LED139, LED139 to LED140, LED140 to LED141, LED141 to LED142, LED142 to LED143, LED143 to LED144, LED144 to LED145, LED145 to LED146, LED146 to LED147, LED147 to LED148, LED148 to LED149, LED149 to LED150, LED150 to LED151, LED151 to LED152, LED152 to LED153, LED153 to LED154, LED154 to LED155, LED155 to LED156, LED156 to LED157, LED157 to LED158, LED158 to LED159, LED159 to LED160, LED160 to LED161, LED161 to LED162, LED162 to LED163, LED163 to LED164, LED164 to LED165, LED165 to LED166, LED166 to LED167, LED167 to LED168, LED168 to LED169, LED169 to LED170, LED170 to LED171, LED171 to LED172, LED172 to LED173, LED173 to LED174, LED174 to LED175, LED175 to LED176, LED176 to LED177, LED177 to LED178, LED178 to LED179, LED179 to LED180, LED180 to LED181, LED181 to LED182, LED182 to LED183, LED183 to LED184, LED184 to LED185

Commit message: WIP
Parts:
- LED101: value LED -> Red_LED

Commit message: I think we are ready
Parts:
- renumbered LED102 to LED101, LED103 to LED102, LED104 to LED103, LED105 to LED104, LED106 to LED105, LED107 to LED106, LED108 to LED107, LED109 to LED108, LED110 to LED109, LED111 to LED110, LED112 to LED111, LED113 to LED112, LED114 to LED113, LED115 to LED114, LED116 to LED115, LED117 to LED116, LED118 to LED117, LED119 to LED118, LED120 to LED119, LED121 to LED120, LED122 to LED121, LED123 to LED122, LED124 to LED123, LED125 to LED124, LED126 to LED125, LED127 to LED126, LED128 to LED127, LED129 to LED128, LED130 to LED129, LED131 to LED130, LED132 to LED131, LED133 to LED132, LED134 to LED133, LED135 to LED134, LED136 to LED135, LED137 to LED136, LED138 to LED137, LED139 to LED138, LED140 to LED139, LED141 to LED140, LED142 to LED141, LED143 to LED142, LED144 to LED143, LED145 to LED144, LED146 to LED145, LED147 to LED146, LED148 to LED147, LED149 to LED148, LED150 to LED149, LED151 to LED150, LED152 to LED151, LED153 to LED152, LED154 to LED153, LED155 to LED154, LED156 to LED155, LED157 to LED156, LED158 to LED157, LED159 to LED158, LED160 to LED159, LED161 to LED160, LED162 to LED161, LED163 to LED162, LED164 to LED163, LED165 to LED164, LED166 to LED165, LED167 to LED166, LED168 to LED167, LED169 to LED168, LED170 to LED169, LED171 to LED170, LED172 to LED171, LED173 to LED172, LED174 to LED173, LED175 to LED174, LED176 to LED175, LED177 to LED176, LED178 to LED177, LED179 to LED178, LED180 to LED179, LED181 to LED180, LED182 to LED181, LED183 to LED182, LED184 to LED183, LED185 to LED184, LED101 to LED2
