File: matrix.sch (KiCad schematic (older format))
At the start: 149 parts

Commit message: WIP
Parts:
- removed D1, D10, D11, D12, D13, D14, D15, D16, D17, D18, D19, D2, D20, D21, D22, D23, D24, D25, D26, D27, D28, D29, D3, D30, D31, D32, D33, D34, D35, D36, D37, D38, D39, D4, D40, D41, D42, D43, D44, D45, D46, D47, D48, D49, D50, D51, D52, D53, D54, D55, D56, D57, D58, D59, D6, D60, D61, D62, D63, D64, D65, D7, D8, D9: 1N4148, 0805:0805D, symbol Device:D
- added D101, D102, D104, D105, D107, D108, D110, D111, D112, D113, D114, D115, D117, D118, D119, D120, D121, D122, D123, D124, D126, D127, D129, D130, D132, D133, D135, D136: D_x2_KCom_AAK, Package_TO_SOT_SMD:SOT-23, symbol Device:D_x2_KCom_AAK
- added D106, D109, D116, D125, D128, D131, D134, D137: D, Diode_SMD:D_SOT-23_ANK, symbol Device:D
- D103: renamed from D5; value 1N4148 -> D; footprint 0805:0805D -> Diode_SMD:D_SOT-23_ANK; Product CD4148WS(0805C) -> (none); Supplier TME -> (none); Supplier Symbol 1N4148-0805 -> (none); Vendor DC Components -> (none)
- renumbered S1 to S101, S2 to S102, S3 to S103, S4 to S104, S5 to S105, S6 to S106, S7 to S107, S8 to S108, S9 to S109, S10 to S110, S11 to S111, S12 to S112, S13 to S113, S14 to S114, S15 to S115, S16 to S116, S17 to S117, S18 to S118, S19 to S119, S20 to S120, S21 to S121, S22 to S122, S23 to S123, S24 to S124, S25 to S125, S26 to S126, S27 to S127, S28 to S128, S29 to S129, S30 to S130, S31 to S131, S32 to S132, S33 to S133, S36 to S134, S34 to S135, S35 to S136, S37 to S137, S38 to S138, S39 to S139, S40 to S140, S41 to S141, S42 to S142, S43 to S143, S44 to S144, S45 to S145, S46 to S146, S47 to S147, S48 to S148, S49 to S149, S50 to S150, S51 to S151, S52 to S152, S53 to S153, S54 to S154, S55 to S155, S56 to S156, S57 to S157, S58 to S158, S59 to S159, S60 to S160, S61 to S161, S62 to S162, S63 to S163, S64 to S164, S65 to S165, S66 to S166, S67 to S167, S68 to S168, S69 to S169, S70 to S170, S71 to S171, S72 to S172, S73 to S173, S74 to S174, S75 to S175, S76 to S176, S77 to S177, S78 to S178, S79 to S179, S80 to S180, S81 to S181, S82 to S182, S83 to S183, S84 to S184
Connections:
- wire segments 663 -> 485
Other:
- note added: "Use BAS70-05 for diodes"

Commit message: finally completed?
Changed lines of the file:
@@
 EESchema Schematic File Version 4
-LIBS:power
 LIBS:mx1a-simple
 LIBS:aker
@@
 U 1 1 5040E2D0
 P 11750 7350
-F 0 "S171" H 11600 7600 60  0000 C CNN
+F 0 "S171" H 11900 7600 60  0000 C CNN
 F 1 "MX1A" H 11750 7450 60  0000 C CNN
 F 2 "mx1a:MX1A_no3d" H 11750 7350 60  0001 C CNN
 F 3 "" H 11750 7350 60  0001 C CNN
 	1    11750 7350
-	1    0    0    -1
+	-1   0    0    -1
 $EndComp
 $Comp
@@
 U 1 1 5040FAF4
 P 6850 8850
-F 0 "S135" H 6700 9100 60  0000 C CNN
+F 0 "S135" H 7000 9100 60  0000 C CNN
 F 1 "MX1A" H 6850 8950 60  0000 C CNN
 F 2 "mx1a:MX1A_no3d" H 6850 8850 60  0001 C CNN
 F 3 "" H 6850 8850 60  0001 C CNN
 	1    6850 8850
-	1    0    0    -1
+	-1   0    0    -1
 $EndComp
 $Comp
@@
 U 1 1 5040DEFF
 P 11750 7050
-F 0 "S170" H 11600 7300 60  0000 C CNN
+F 0 "S170" H 11900 7300 60  0000 C CNN
 F 1 "MX1A" H 11750 7150 60  0000 C CNN
 F 2 "mx1a:MX1A_no3d" H 11750 7050 60  0001 C CNN
 F 3 "" H 11750 7050 60  0001 C CNN
 	1    11750 7050
-	1    0    0    -1
+	-1   0    0    -1
 $EndComp
 $Comp
@@
 U 1 1 5051FE50
 P 12450 7350
-F 0 "S181" H 12600 7600 60  0000 C CNN
+F 0 "S181" H 12300 7600 60  0000 C CNN
 F 1 "MX1A" H 12450 7450 60  0000 C CNN
 F 2 "mx1a:MX1A_no3d" H 12450 7350 60  0001 C CNN
 F 3 "" H 12450 7350 60  0001 C CNN
 	1    12450 7350
-	-1   0    0    -1
+	1    0    0    -1
 $EndComp
 $Comp
@@
 U 1 1 5B6C3490
 P 3400 3950
-F 0 "D101" V 3200 3900 50  0000 R BNN
+F 0 "D101" V 3150 3900 50  0000 R TNN
 F 1 "D_x2_KCom_AAK" V 3355 4029 50  0001 L CNN
 F 2 "Package_TO_SOT_SMD:SOT-23" H 3400 3950 50  0001 C CNN
@@
 U 1 1 5C200A9A
 P 4100 3950
-F 0 "D104" V 4300 3900 50  0000 R TNN
+F 0 "D104" V 3850 3900 50  0000 R TNN
 F 1 "D_x2_KCom_AAK" V 4055 4029 50  0001 L CNN
 F 2 "Package_TO_SOT_SMD:SOT-23" H 4100 3950 50  0001 C CNN
 F 3 "~" H 4100 3950 50  0001 C CNN
 	1    4100 3950
-	0    -1   -1   0
+	0    -1   1    0
 $EndComp
 Wire Wire Line
@@
 U 1 1 5C269BB2
 P 4800 3950
-F 0 "D107" V 5000 3900 50  0000 R TNN
+F 0 "D107" V 4550 3900 50  0000 R TNN
 F 1 "D_x2_KCom_AAK" V 4755 4029 50  0001 L CNN
 F 2 "Package_TO_SOT_SMD:SOT-23" H 4800 3950 50  0001 C CNN
 F 3 "~" H 4800 3950 50  0001 C CNN
 	1    4800 3950
-	0    -1   -1   0
+	0    -1   1    0
 $EndComp
 Wire Wire Line
@@
 U 1 1 5C3A572D
 P 5500 3950
-F 0 "D110" V 5700 3900 50  0000 R TNN
+F 0 "D110" V 5250 3900 50  0000 R TNN
 F 1 "D_x2_KCom_AAK" V 5455 4029 50  0001 L CNN
 F 2 "Package_TO_SOT_SMD:SOT-23" H 5500 3950 50  0001 C CNN
 F 3 "~" H 5500 3950 50  0001 C CNN
 	1    5500 3950
-	0    -1   -1   0
+	0    -1   1    0
 $EndComp
 Wire Wire Line
@@
 U 1 1 5C478F5A
 P 6900 3950
-F 0 "D114" V 7100 3900 50  0000 R TNN
+F 0 "D114" V 6650 3900 50  0000 R TNN
 F 1 "D_x2_KCom_AAK" V 6855 4029 50  0001 L CNN
 F 2 "Package_TO_SOT_SMD:SOT-23" H 6900 3950 50  0001 C CNN
 F 3 "~" H 6900 3950 50  0001 C CNN
 	1    6900 3950
-	0    -1   -1   0
+	0    -1   1    0
 $EndComp
 Wire Wire Line
@@
 F 3 "~" H 7600 3950 50  0001 C CNN
 	1    7600 3950
-	0    -1   -1   0
+	0    -1   1    0
 $EndComp
 Wire Wire Line
@@
 F 3 "~" H 8300 3950 50  0001 C CNN
 	1    8300 3950
-	0    -1   -1   0
+	0    -1   1    0
 $EndComp
 Wire Wire Line
@@
 F 3 "~" H 9000 3950 50  0001 C CNN
 	1    9000 3950
-	0    -1   -1   0
+	0    -1   1    0
 $EndComp
 Wire Wire Line
@@
 F 3 "~" H 9700 3950 50  0001 C CNN
 	1    9700 3950
-	0    -1   -1   0
+	0    -1   1    0
 $EndComp
 Wire Wire Line
@@
 F 3 "~" H 10400 3950 50  0001 C CNN
 	1    10400 3950
-	0    -1   -1   0
+	0    -1   1    0
 $EndComp
 Wire Wire Line
@@
 F 3 "~" H 11100 3950 50  0001 C CNN
 	1    11100 3950
-	0    -1   -1   0
+	0    -1   1    0
 $EndComp
 Wire Wire Line
@@
 F 3 "~" H 11800 3950 50  0001 C CNN
 	1    11800 3950
-	0    -1   -1   0
+	0    -1   1    0
 $EndComp
 Wire Wire Line
@@
 F 3 "~" H 12500 3950 50  0001 C CNN
 	1    12500 3950
-	0    -1   -1   0
+	0    -1   1    0
 $EndComp
 Wire Wire Line
@@
 	8500 1400 8500 3950
 Wire Wire Line
-	4300 1400 4300 3950
-Wire Wire Line
 	5000 1400 5000 3950
 Wire Wire Line
 	5700 1400 5700 3950
-Wire Wire Line
-	7100 1400 7100 3950
 Wire Wire Line
 	7800 1400 7800 3950
@@
 Wire Wire Line
 	4250 6500 4250 6900
-Connection ~ 4300 3950
-Wire Wire Line
-	4300 3950 4300 6050
 Connection ~ 5000 3950
 Wire Wire Line
@@
 	12700 3950 12700 6450
 Connection ~ 12000 3950
-Wire Wire Line
-	12000 3950 12000 6050
 Connection ~ 11300 3950
 Wire Wire Line
@@
 Wire Wire Line
 	7800 3950 7800 6050
-Connection ~ 7100 3950
-Wire Wire Line
-	7100 3950 7100 6050
 Wire Wire Line
 	6400 3950 6400 6050
@@
 F 3 "~" H 11800 6050 50  0001 C CNN
 	1    11800 6050
-	0    -1   1    0
+	0    -1   -1   0
 $EndComp
 Wire Wire Line
@@
 Wire Wire Line
 	11950 6500 11950 6900
-Connection ~ 12000 6050
 Connection ~ 11300 6050
 Connection ~ 10600 6050
@@
 $EndComp
 Wire Wire Line
-	12000 6050 12000 9150
-Wire Wire Line
 	11950 8700 11950 8850
 Wire Wire Line
@@
 Wire Wire Line
 	3600 3950 3600 6450
+Connection ~ 11950 6900
+Wire Wire Line
+	4300 1400 4300 3950
+Connection ~ 4300 3950
+Wire Wire Line
+	4300 3950 4300 6050
+Connection ~ 7100 3950
+Wire Wire Line
+	7100 3950 7100 6050
+Wire Wire Line
+	7100 1400 7100 3950
+Wire Wire Line
+	12000 3950 12000 6050
+Connection ~ 12000 6050
+Wire Wire Line
+	12000 6050 12000 9150
 $EndSCHEMATC

Commit message: WIP
Parts:
- D101, D102, D104, D105, D107, D108, D110, D111, D112, D113, D114, D115, D117, D118, D119, D120, D121, D122, D123, D124, D126, D127, D129, D130, D132, D133, D135, D136: value D_x2_KCom_AAK -> BAS70-05
- D103, D106, D109, D116, D125, D128, D131, D134, D137: value D -> BAS70-05
