File: mechanical.sch (KiCad schematic (older format))
At the start: 21 parts

Commit message: WIP
Parts:
- MK1, MK2, MK3, MK4, MK5, MK6, MXST1, MXST10, MXST11, MXST12, MXST13, MXST14, MXST15, MXST2, MXST3, MXST4, MXST5, MXST6, MXST7, MXST8, MXST9: symbol Mechanical:Mounting_Hole -> Mechanical:MountingHole
Changed lines of the file:
@@
 EESchema Schematic File Version 4
-LIBS:keyboard-cache
 EELAYER 26 0
 EELAYER END
@@
 $EndDescr
 $Comp
-L Mechanical:Mounting_Hole MK1
+L Mechanical:MountingHole MK1
 U 1 1 5B8D09B9
 P 2000 2000
@@
 $EndComp
 $Comp
-L Mechanical:Mounting_Hole MK2
+L Mechanical:MountingHole MK2
 U 1 1 5B8D09D3
 P 2000 2300
@@
 $EndComp
 $Comp
-L Mechanical:Mounting_Hole MK3
+L Mechanical:MountingHole MK3
 U 1 1 5B8D09EF
 P 2000 2600
@@
 $EndComp
 $Comp
-L Mechanical:Mounting_Hole MK4
+L Mechanical:MountingHole MK4
 U 1 1 5B8D0A0F
 P 2000 2900
@@
 $EndComp
 $Comp
-L Mechanical:Mounting_Hole MK5
+L Mechanical:MountingHole MK5
 U 1 1 5B8D0A2D
 P 2000 3200
@@
 $EndComp
 $Comp
-L Mechanical:Mounting_Hole MK6
+L Mechanical:MountingHole MK6
 U 1 1 5B9103CB
 P 2000 3500
@@
 $EndComp
 $Comp
-L Mechanical:Mounting_Hole MXST1
+L Mechanical:MountingHole MXST1
 U 1 1 5B91076A
 P 4000 2000
@@
 $EndComp
 $Comp
-L Mechanical:Mounting_Hole MXST2
+L Mechanical:MountingHole MXST2
 U 1 1 5B910A3A
 P 4000 2300
@@
 $EndComp
 $Comp
-L Mechanical:Mounting_Hole MXST3
+L Mechanical:MountingHole MXST3
 U 1 1 5B910A80
 P 4000 2600
@@
 $EndComp
 $Comp
-L Mechanical:Mounting_Hole MXST4
+L Mechanical:MountingHole MXST4
 U 1 1 5B910AAA
 P 4000 2900
@@
 $EndComp
 $Comp
-L Mechanical:Mounting_Hole MXST5
+L Mechanical:MountingHole MXST5
 U 1 1 5B910AD6
 P 4000 3200
@@
 $EndComp
 $Comp
-L Mechanical:Mounting_Hole MXST6
+L Mechanical:MountingHole MXST6
 U 1 1 5B910B0E
 P 4000 3500
@@
 $EndComp
 $Comp
-L Mechanical:Mounting_Hole MXST7
+L Mechanical:MountingHole MXST7
 U 1 1 5B910B42
 P 4000 3800
@@
 $EndComp
 $Comp
-L Mechanical:Mounting_Hole MXST8
+L Mechanical:MountingHole MXST8
 U 1 1 5B910B74
 P 4000 4100
@@
 $EndComp
 $Comp
-L Mechanical:Mounting_Hole MXST9
+L Mechanical:MountingHole MXST9
 U 1 1 5B910C03
 P 4000 4400
@@
 $EndComp
 $Comp
-L Mechanical:Mounting_Hole MXST10
+L Mechanical:MountingHole MXST10
 U 1 1 5B910D01
 P 4000 4700
@@
 $EndComp
 $Comp
-L Mechanical:Mounting_Hole MXST11
+L Mechanical:MountingHole MXST11
 U 1 1 5B910DB9
 P 4000 5000
@@
 $EndComp
 $Comp
-L Mechanical:Mounting_Hole MXST12
+L Mechanical:MountingHole MXST12
 U 1 1 5B910DF7
 P 4000 5300
@@
 $EndComp
 $Comp
-L Mechanical:Mounting_Hole MXST13
+L Mechanical:MountingHole MXST13
 U 1 1 5B910E37
 P 4000 5600
@@
 $EndComp
 $Comp
-L Mechanical:Mounting_Hole MXST14
+L Mechanical:MountingHole MXST14
 U 1 1 5B910E75
 P 4000 5900
@@
 $EndComp
 $Comp
-L Mechanical:Mounting_Hole MXST15
+L Mechanical:MountingHole MXST15
 U 1 1 5B910EED
 P 4000 6200

Commit message: WIP
Parts:
- MXST1, MXST10, MXST11, MXST12, MXST13, MXST14, MXST15, MXST2, MXST3, MXST4, MXST5, MXST6, MXST7, MXST8, MXST9: value Stabilizer_Mounting -> Cherry_Stabilizer
Changed lines of the file:
@@
 F 1 "Mounting_Hole" H 2100 1955 50  0000 L CNN
 F 2 "hole:PKRHSL" H 2000 2000 50  0001 C CNN
-F 3 "" H 2000 2000 50  0001 C CNN
+F 3 "~" H 2000 2000 50  0001 C CNN
 	1    2000 2000
 	1    0    0    -1
@@
 F 1 "Mounting_Hole" H 2100 2255 50  0000 L CNN
 F 2 "hole:PKRHC" H 2000 2300 50  0001 C CNN
-F 3 "" H 2000 2300 50  0001 C CNN
+F 3 "~" H 2000 2300 50  0001 C CNN
 	1    2000 2300
 	1    0    0    -1
@@
 F 1 "Mounting_Hole" H 2100 2555 50  0000 L CNN
 F 2 "hole:PKRH" H 2000 2600 50  0001 C CNN
-F 3 "" H 2000 2600 50  0001 C CNN
+F 3 "~" H 2000 2600 50  0001 C CNN
 	1    2000 2600
 	1    0    0    -1
@@
 F 1 "Mounting_Hole" H 2100 2855 50  0000 L CNN
 F 2 "hole:PKRH" H 2000 2900 50  0001 C CNN
-F 3 "" H 2000 2900 50  0001 C CNN
+F 3 "~" H 2000 2900 50  0001 C CNN
 	1    2000 2900
 	1    0    0    -1
@@
 F 1 "Mounting_Hole" H 2100 3155 50  0000 L CNN
 F 2 "hole:PKRH" H 2000 3200 50  0001 C CNN
-F 3 "" H 2000 3200 50  0001 C CNN
+F 3 "~" H 2000 3200 50  0001 C CNN
 	1    2000 3200
 	1    0    0    -1
@@
 F 1 "Mounting_Hole" H 2100 3455 50  0000 L CNN
 F 2 "hole:PKRHSL" H 2000 3500 50  0001 C CNN
-F 3 "" H 2000 3500 50  0001 C CNN
+F 3 "~" H 2000 3500 50  0001 C CNN
 	1    2000 3500
 	1    0    0    -1
@@
 P 4000 2000
 F 0 "MXST1" H 4100 2046 50  0000 L CNN
-F 1 "Stabilizer_Mounting" H 4100 1955 50  0000 L CNN
+F 1 "Cherry_Stabilizer" H 4100 1955 50  0000 L CNN
 F 2 "mx1a:MXST" H 4000 2000 50  0001 C CNN
-F 3 "" H 4000 2000 50  0001 C CNN
+F 3 "~" H 4000 2000 50  0001 C CNN
 	1    4000 2000
 	1    0    0    -1
@@
 P 4000 2300
 F 0 "MXST2" H 4100 2346 50  0000 L CNN
-F 1 "Stabilizer_Mounting" H 4100 2255 50  0000 L CNN
+F 1 "Cherry_Stabilizer" H 4100 2255 50  0000 L CNN
 F 2 "mx1a:MXST" H 4000 2300 50  0001 C CNN
-F 3 "" H 4000 2300 50  0001 C CNN
+F 3 "~" H 4000 2300 50  0001 C CNN
 	1    4000 2300
 	1    0    0    -1
@@
 P 4000 2600
 F 0 "MXST3" H 4100 2646 50  0000 L CNN
-F 1 "Stabilizer_Mounting" H 4100 2555 50  0000 L CNN
+F 1 "Cherry_Stabilizer" H 4100 2555 50  0000 L CNN
 F 2 "mx1a:MXST" H 4000 2600 50  0001 C CNN
-F 3 "" H 4000 2600 50  0001 C CNN
+F 3 "~" H 4000 2600 50  0001 C CNN
 	1    4000 2600
 	1    0    0    -1
@@
 P 4000 2900
 F 0 "MXST4" H 4100 2946 50  0000 L CNN
-F 1 "Stabilizer_Mounting" H 4100 2855 50  0000 L CNN
+F 1 "Cherry_Stabilizer" H 4100 2855 50  0000 L CNN
 F 2 "mx1a:MXST" H 4000 2900 50  0001 C CNN
-F 3 "" H 4000 2900 50  0001 C CNN
+F 3 "~" H 4000 2900 50  0001 C CNN
 	1    4000 2900
 	1    0    0    -1
@@
 P 4000 3200
 F 0 "MXST5" H 4100 3246 50  0000 L CNN
-F 1 "Stabilizer_Mounting" H 4100 3155 50  0000 L CNN
+F 1 "Cherry_Stabilizer" H 4100 3155 50  0000 L CNN
 F 2 "mx1a:MXST" H 4000 3200 50  0001 C CNN
-F 3 "" H 4000 3200 50  0001 C CNN
+F 3 "~" H 4000 3200 50  0001 C CNN
 	1    4000 3200
 	1    0    0    -1
@@
 P 4000 3500
 F 0 "MXST6" H 4100 3546 50  0000 L CNN
-F 1 "Stabilizer_Mounting" H 4100 3455 50  0000 L CNN
+F 1 "Cherry_Stabilizer" H 4100 3455 50  0000 L CNN
 F 2 "mx1a:MXST" H 4000 3500 50  0001 C CNN
-F 3 "" H 4000 3500 50  0001 C CNN
+F 3 "~" H 4000 3500 50  0001 C CNN
 	1    4000 3500
 	1    0    0    -1
@@
 P 4000 3800
 F 0 "MXST7" H 4100 3846 50  0000 L CNN
-F 1 "Stabilizer_Mounting" H 4100 3755 50  0000 L CNN
+F 1 "Cherry_Stabilizer" H 4100 3755 50  0000 L CNN
 F 2 "mx1a:MXST" H 4000 3800 50  0001 C CNN
-F 3 "" H 4000 3800 50  0001 C CNN
+F 3 "~" H 4000 3800 50  0001 C CNN
 	1    4000 3800
 	1    0    0    -1
@@
 P 4000 4100
 F 0 "MXST8" H 4100 4146 50  0000 L CNN
-F 1 "Stabilizer_Mounting" H 4100 4055 50  0000 L CNN
+F 1 "Cherry_Stabilizer" H 4100 4055 50  0000 L CNN
 F 2 "mx1a:MXST" H 4000 4100 50  0001 C CNN
-F 3 "" H 4000 4100 50  0001 C CNN
+F 3 "~" H 4000 4100 50  0001 C CNN
 	1    4000 4100
 	1    0    0    -1
@@
 P 4000 4400
 F 0 "MXST9" H 4100 4446 50  0000 L CNN
-F 1 "Stabilizer_Mounting" H 4100 4355 50  0000 L CNN
+F 1 "Cherry_Stabilizer" H 4100 4355 50  0000 L CNN
 F 2 "mx1a:MXST" H 4000 4400 50  0001 C CNN
-F 3 "" H 4000 4400 50  0001 C CNN
+F 3 "~" H 4000 4400 50  0001 C CNN
 	1    4000 4400
 	1    0    0    -1
@@
 P 4000 4700
 F 0 "MXST10" H 4100 4746 50  0000 L CNN
-F 1 "Stabilizer_Mounting" H 4100 4655 50  0000 L CNN
+F 1 "Cherry_Stabilizer" H 4100 4655 50  0000 L CNN
 F 2 "mx1a:MXST" H 4000 4700 50  0001 C CNN
-F 3 "" H 4000 4700 50  0001 C CNN
+F 3 "~" H 4000 4700 50  0001 C CNN
 	1    4000 4700
 	1    0    0    -1
@@
 P 4000 5000
 F 0 "MXST11" H 4100 5046 50  0000 L CNN
-F 1 "Stabilizer_Mounting" H 4100 4955 50  0000 L CNN
+F 1 "Cherry_Stabilizer" H 4100 4955 50  0000 L CNN
 F 2 "mx1a:MXST" H 4000 5000 50  0001 C CNN
-F 3 "" H 4000 5000 50  0001 C CNN
+F 3 "~" H 4000 5000 50  0001 C CNN
 	1    4000 5000
 	1    0    0    -1
@@
 P 4000 5300
 F 0 "MXST12" H 4100 5346 50  0000 L CNN
-F 1 "Stabilizer_Mounting" H 4100 5255 50  0000 L CNN
+F 1 "Cherry_Stabilizer" H 4100 5255 50  0000 L CNN
 F 2 "mx1a:MXST" H 4000 5300 50  0001 C CNN
-F 3 "" H 4000 5300 50  0001 C CNN
+F 3 "~" H 4000 5300 50  0001 C CNN
 	1    4000 5300
 	1    0    0    -1
@@
 P 4000 5600
 F 0 "MXST13" H 4100 5646 50  0000 L CNN
-F 1 "Stabilizer_Mounting" H 4100 5555 50  0000 L CNN
+F 1 "Cherry_Stabilizer" H 4100 5555 50  0000 L CNN
 F 2 "mx1a:MXST" H 4000 5600 50  0001 C CNN
-F 3 "" H 4000 5600 50  0001 C CNN
+F 3 "~" H 4000 5600 50  0001 C CNN
 	1    4000 5600
 	1    0    0    -1
@@
 P 4000 5900
 F 0 "MXST14" H 4100 5946 50  0000 L CNN
-F 1 "Stabilizer_Mounting" H 4100 5855 50  0000 L CNN
+F 1 "Cherry_Stabilizer" H 4100 5855 50  0000 L CNN
 F 2 "mx1a:MXST" H 4000 5900 50  0001 C CNN
-F 3 "" H 4000 5900 50  0001 C CNN
+F 3 "~" H 4000 5900 50  0001 C CNN
 	1    4000 5900
 	1    0    0    -1
@@
 P 4000 6200
 F 0 "MXST15" H 4100 6246 50  0000 L CNN
-F 1 "Stabilizer_Mounting" H 4100 6155 50  0000 L CNN
+F 1 "Cherry_Stabilizer" H 4100 6155 50  0000 L CNN
 F 2 "mx1a:MXST" H 4000 6200 50  0001 C CNN
-F 3 "" H 4000 6200 50  0001 C CNN
+F 3 "~" H 4000 6200 50  0001 C CNN
 	1    4000 6200
 	1    0    0    -1
